Commit message: fix material warning

File: ros/src/diffbot_description/urdf/wheel.urdf.xacro (robot description, xacro)
@@ -23,5 +23,5 @@
           <cylinder length="${width}" radius="${radius}" />
         </geometry>
-        <material name="DarkGray" />
+        <material name="black" />
       </visual>
       <collision>
@@ -59,5 +59,5 @@
       <joint name="${fb}_${lr}_wheel_joint" />
       <actuator name="${fb}_${lr}_wheel_joint_motor">
-        <hardwareInterface>EffortJointInterface</hardwareInterface>
+        <hardwareInterface>VelocityJointInterface</hardwareInterface>
         <mechanicalReduction>1</mechanicalReduction>
       </actuator>

Commit message: update robot description and add control package

File: ros/src/diffbot_description/urdf/wheel.urdf.xacro (robot description, xacro)
@@ -57,7 +57,9 @@
     <transmission name="${fb}_${lr}_wheel_joint_trans">
       <type>transmission_interface/SimpleTransmission</type>
-      <joint name="${fb}_${lr}_wheel_joint" />
+      <joint name="${fb}_${lr}_wheel_joint">
+        <hardwareInterface>hardware_interface/VelocityJointInterface</hardwareInterface>
+      </joint>
       <actuator name="${fb}_${lr}_wheel_joint_motor">
-        <hardwareInterface>VelocityJointInterface</hardwareInterface>
+        <hardwareInterface>hardware_interface/VelocityJointInterface</hardwareInterface>
         <mechanicalReduction>1</mechanicalReduction>
       </actuator>

Commit message: fix robot description using vscode prview

File: ros/src/diffbot_description/urdf/wheel.urdf.xacro (robot description, xacro)
@@ -19,5 +19,5 @@
     <link name="${fb}_${lr}_wheel">
       <visual>
-        <origin xyz="0 0 0" rpy="${flipY*M_PI/2} 0  0 " />
+        <origin xyz="0 0 0" rpy="${flipY*M_PI/2} 0 0 " />
         <geometry>
           <cylinder length="${width}" radius="${radius}" />
@@ -50,5 +50,5 @@
       <child link="${fb}_${lr}_wheel"/>
       <origin xyz="${transX} ${reflect * (transY + wheel_width/2.0)} ${transZ}" rpy="0 0 0" />
-      <axis xyz="0 1 0" rpy="0  0" />
+      <axis xyz="0 1 0" rpy="0 0 0" />
       <limit effort="100" velocity="100"/>
       <joint_properties damping="0.0" friction="0.0"/>

Commit message: fix inertia matrix

File: ros/src/diffbot_description/urdf/wheel.urdf.xacro (robot description, xacro)
@@ -2,7 +2,7 @@
 <robot name="wheel" xmlns:xacro="http://www.ros.org/wiki/xacro">
   <xacro:macro name="cylinder_inertia" params="m r h">
-    <inertia  ixx="${m*(3*r*r+h*h)/12}" ixy = "0" ixz = "0"
-              iyy="${m*(3*r*r+h*h)/12}" iyz = "0"
-              izz="${m*r*r/2}" />
+    <inertia  ixx="${m/12*(3*r*r+h*h)}" ixy = "0" ixz = "0"
+              iyy="${m/2*(r*r)}" iyz = "0"
+              izz="${m/12*(3*r*r+h*h)}" />
   </xacro:macro>
   <!--fb : front, back ; lr: left, right -->
@@ -33,5 +33,5 @@
       <inertial>
         <mass value="${mass}" />
-        <origin xyz="0 0 0" />
+        <!--origin xyz="0 0 0" /-->
         <xacro:cylinder_inertia  m="${mass}" r="${radius}" h="${width}" />
       </inertial>

Commit message: using default pi macro for wheel macro

File: ros/src/diffbot_description/urdf/wheel.urdf.xacro (robot description, xacro)
@@ -19,5 +19,5 @@
     <link name="${fb}_${lr}_wheel">
       <visual>
-        <origin xyz="0 0 0" rpy="${flipY*M_PI/2} 0 0 " />
+        <origin xyz="0 0 0" rpy="${flipY*pi_2} 0 0 " />
         <geometry>
           <cylinder length="${width}" radius="${radius}" />
@@ -26,5 +26,5 @@
       </visual>
       <collision>
-        <origin xyz="0 0 0" rpy="${flipY*M_PI/2} 0 0 " />
+        <origin xyz="0 0 0" rpy="${flipY*pi_2} 0 0 " />
         <geometry>
           <cylinder length="${width}" radius="${radius}" />
