Commit message: fix caster wheel inertias

File: ros/src/diffbot_description/urdf/caster_wheel.urdf.xacro (robot description, xacro)
@@ -14,8 +14,7 @@
         <link name="${locationprefix}_caster_rotation_link">
             <inertial>
-            <!-- <origin xyz="0 0 -0.042500000044" rpy="${0.5 * pi} ${24 * deg_to_rad} ${1.5 * pi}" /> -->
-                <origin xyz="0 0 0" rpy="${24 * deg_to_rad} 0 ${0.5 * pi} " />
-                <mass value="0.3097539019" />
-                <xacro:box_inertia  m="${base_mass}" l="${base_length}" w="${base_width}" h="${base_height}" />
+                <origin xyz="0 0 ${-caster_base_size/2.0}" rpy="0 0 0" />
+                <mass value="${caster_base_mass}" />
+                <xacro:box_inertia  m="${caster_base_mass}" l="${caster_base_size}" w="${caster_base_size}" h="${caster_base_size}" />
             </inertial>
             <visual>
@@ -47,5 +46,5 @@
         <link name="${locationprefix}_caster_wheel_link">
             <xacro:cylinder_inertial mass="${caster_wheel_mass}" radius="${caster_wheel_radius}" length="${caster_wheel_width}">
-            <origin xyz="0 0 0" rpy="${0.5 * pi} 0 0" />
+                <origin xyz="0 0 0" rpy="${pi_2} 0 0" />
             </xacro:cylinder_inertial>
             <visual>

Commit message: use meshes for difbot model

File: ros/src/diffbot_description/urdf/caster_wheel.urdf.xacro (robot description, xacro)
@@ -4,4 +4,36 @@
     <xacro:macro name="caster_wheel" params="locationprefix locationright wheel_base_dx
         flipY:=${1}">
+        <joint name="${locationprefix}_caster_base_joint" type="fixed">
+            <origin xyz="${wheel_base_dx} ${-caster_wheel_base_dy * locationright} ${caster_wheel_base_dz}" rpy="0 0 0" />
+            <parent link="base_link" />
+            <child link="${locationprefix}_caster_base_link" />
+            <axis xyz="0 0 1" />
+            <dynamics damping="0.01" friction="0.0"/>
+        </joint>
+        <link name="${locationprefix}_caster_base_link">
+            <inertial>
+                <origin xyz="0 0 ${-caster_base_size/2.0}" rpy="0 0 0" />
+                <mass value="${caster_base_mass}" />
+                <xacro:box_inertia  m="${caster_base_mass}" l="${caster_base_size}" w="${caster_base_size}" h="${caster_base_size}" />
+            </inertial>
+            <visual>
+                <origin xyz="0 0 ${-caster_base_size/2.0}" rpy="0 0 0" />
+                <geometry>
+                    <mesh filename="package://diffbot_description/meshes/caster_base.stl" />
+                    <box size="${caster_base_size} ${caster_base_size} ${caster_base_size}" />
+                </geometry>
+                <xacro:insert_block name="material_silver" />
+            </visual>
+            <collision>
+                <origin xyz="0 0 ${-caster_base_size/2.0}" rpy="0 0 0" />
+                <geometry>
+                    <!--mesh filename="package://mir_description/meshes/collision/caster_wheel_base.stl" /-->
+                    <box size="${caster_base_size} ${caster_base_size} ${caster_base_size}" />
+                </geometry>
+            </collision>
+        </link>
+        <gazebo reference="${locationprefix}_caster_base_link">
+            <material>Gazebo/Grey</material>
+        </gazebo>
         <!-- caster hub -->
         <joint name="${locationprefix}_caster_rotation_joint" type="continuous">
@@ -21,6 +53,6 @@
                 <origin xyz="0 0 ${-caster_base_size/2.0}" rpy="0 0 0" />
                 <geometry>
-                    <!--mesh filename="package://mir_description/meshes/visual/caster_wheel_base.stl" /-->
-                    <box size="${caster_base_size} ${caster_base_size} ${caster_base_size}" />
+                    <mesh filename="package://diffbot_description/meshes/caster_wheel_support.stl" />
+                    <!--box size="${caster_base_size} ${caster_base_size} ${caster_base_size}" /-->
                 </geometry>
                 <xacro:insert_block name="material_silver" />
@@ -49,8 +81,8 @@
             </xacro:cylinder_inertial>
             <visual>
-                <origin xyz="0 0 0" rpy="${flipY*pi_2} 0 0" />
+                <origin xyz="0 0 0" rpy="0 0 0" />
                 <geometry>
-                    <!--mesh filename="package://mir_description/meshes/visual/wheel.stl" -->
-                    <cylinder length="${caster_wheel_width}" radius="${caster_wheel_radius}" />
+                    <mesh filename="package://diffbot_description/meshes/caster_wheel.stl" />
+                    <!--cylinder length="${caster_wheel_width}" radius="${caster_wheel_radius}" /-->
                 </geometry>
                 <xacro:insert_block name="material_dark_grey" />
@@ -59,5 +91,5 @@
                 <origin xyz="0 0 0" rpy="${flipY*pi_2} 0 0" />
                 <geometry>
-                    <!--mesh filename="package://mir_description/meshes/visual/wheel.stl" -->
+                    <!--mesh filename="package://diffbot_description/meshes/wheel.stl" -->
                     <cylinder length="${caster_wheel_width}" radius="${caster_wheel_radius}" />
                 </geometry>

File: ros/src/diffbot_description/urdf/diffbot.xacro (robot description, xacro)
@@ -4,22 +4,21 @@
   <!--All units in m-kg-s-radians unit system -->
   <!-- Constants for robot dimensions -->
-  <!--xacro:property name="pi" value="3.1415926535897931" /-->
-  <xacro:property name="pi_2" value="1.570796327" />
+  <xacro:property name="pi_2" value="${pi/2.0}" />
   <xacro:property name="deg_to_rad" value="0.017453293" />
   <!-- Main body height, length width and mass -->
   <!-- Main body box base -->
-  <xacro:property name="base_height" value="0.02" />
-  <xacro:property name="base_length" value="0.30" />
-  <xacro:property name="base_width" value="0.15" />
-  <xacro:property name="base_mass" value="16.0" /> <!-- in kg-->
+  <xacro:property name="base_height" value="0.01" />
+  <xacro:property name="base_length" value="0.22" />
+  <xacro:property name="base_width" value="0.11" />
+  <xacro:property name="base_mass" value="0.8" /> <!-- in kg-->
   <!-- Wheel properties -->
   <!-- Wheel radius, width and mass -->
-  <xacro:property name="wheel_radius" value="0.04" />
+  <xacro:property name="wheel_radius" value="0.035" />
   <xacro:property name="wheel_width" value="0.02" />
-  <xacro:property name="wheel_mass" value="1.0" /> <!-- in kg-->
+  <xacro:property name="wheel_mass" value="0.5" /> <!-- in kg-->
   <!-- Wheel placement relative to base origin -->
-  <xacro:property name="base_x_origin_to_wheel_origin" value="${base_length/2.0*0.7}" />
-  <xacro:property name="base_y_origin_to_wheel_origin" value="${base_width/2.0}" />
-  <xacro:property name="base_z_origin_to_wheel_origin" value="0.0" />
+  <xacro:property name="base_x_origin_to_wheel_origin" value="${base_length/2.0*0.15}" />
+  <xacro:property name="base_y_origin_to_wheel_origin" value="${base_width/1.65}" />
+  <xacro:property name="base_z_origin_to_wheel_origin" value="-0.02" />
   <!-- Caster wheel radius, width and mass -->
   <xacro:property name="caster_wheel_width" value="0.01" />
@@ -27,13 +26,13 @@
   <xacro:property name="caster_wheel_mass" value="0.5" /> <!-- in kg-->
   <!-- Caster wheel base size, width and mass -->
-  <xacro:property name="caster_wheel_dx" value="${-caster_base_size/2.0}" />
+  <xacro:property name="caster_wheel_dx" value="${-caster_base_size/2.0*0.8}" />
   <xacro:property name="caster_wheel_dy" value="-1" />
   <xacro:property name="caster_wheel_dz" value="${-caster_base_size}" />
   <!--xacro:property name="front_caster_wheel_base_dx" value="0.341346" /-->
   <xacro:property name="caster_base_mass" value="0.02" />
-  <xacro:property name="caster_base_size" value="0.02" />
-  <xacro:property name="back_caster_wheel_base_dx" value="-0.270154" />
+  <xacro:property name="caster_base_size" value="0.04" />
+  <xacro:property name="back_caster_wheel_base_dx" value="${-base_length/2*0.69}" />
   <xacro:property name="caster_wheel_base_dy" value="0.203" />
-  <xacro:property name="caster_wheel_base_dz" value="${-base_height/2.0}" />
+  <xacro:property name="caster_wheel_base_dz" value="0.002" />
   <!-- Hokuyo Laser scanner -->
   <xacro:property name="hokuyo_size" value="0.05" />
@@ -50,5 +49,5 @@
   <link name="base_footprint">
     <collision>
-        <origin xyz="0 0 0" rpy="0 0 0" />
+        <origin xyz="0 0 ${-base_z_origin_to_wheel_origin}" rpy="0 0 0" />
         <geometry>
             <box size="0.001 0.001 0.001" />
@@ -69,10 +68,11 @@
       <origin xyz="0 0 0" />
       <!--The 3x3 rotational inertia matrix. -->
-      <xacro:box_inertia  m="${base_mass}" l="${base_length}" w="${base_width}" h="${base_height}" />
+      <xacro:box_inertia m="${base_mass}" l="${base_length}" w="${base_width}" h="${base_height}" />
     </inertial>
     <visual>
       <origin xyz="0 0 0" rpy="0 0 0" />
       <geometry>
-          <box size="${base_length} ${base_width} ${base_height}" />
+          <!--box size="${base_length} ${base_width} ${base_height}" /-->
+          <mesh filename="package://diffbot_description/meshes/chassis.stl" />
       </geometry>
       <material name="white" />
@@ -87,5 +87,5 @@
   <!-- Wheel definitions -->
   <xacro:wheel fb="front" lr="right" parent="base_link"
-    mass="${wheel_mass}" radius="${wheel_radius}" width="${wheel_width}" reflect="1"
+    mass="${wheel_mass}" radius="${wheel_radius}" width="${wheel_width}" reflect="-1"
     transX="${base_x_origin_to_wheel_origin}"
     transY="${base_y_origin_to_wheel_origin}"
@@ -93,5 +93,5 @@
     flipY="1" />
   <xacro:wheel fb="front" lr="left" parent="base_link"
-    mass="${wheel_mass}" radius="${wheel_radius}" width="${wheel_width}" reflect="-1"
+    mass="${wheel_mass}" radius="${wheel_radius}" width="${wheel_width}" reflect="1"
     transX="${base_x_origin_to_wheel_origin}"
     transY="${base_y_origin_to_wheel_origin}"
@@ -100,4 +100,4 @@
     <!-- Caster back  -->
     <!-- Joint between base_link and back caster wheel -->
-    <xacro:caster_wheel locationprefix="back" locationright="0" wheel_base_dx="${-base_length/2.0*0.9}" />
+    <xacro:caster_wheel locationprefix="back" locationright="0" wheel_base_dx="${back_caster_wheel_base_dx}" />
 </robot>

File: ros/src/diffbot_description/urdf/wheel.urdf.xacro (robot description, xacro)
@@ -5,4 +5,17 @@
               iyy="${m/2*(r*r)}" iyz = "0"
               izz="${m/12*(3*r*r+h*h)}" />
+  </xacro:macro>
+  <!-- Transmission is important to link the joints and the controller -->
+  <xacro:macro name="transmission" params="joint">
+    <transmission name="${joint}_trans">
+      <type>transmission_interface/SimpleTransmission</type>
+      <joint name="${joint}">
+        <hardwareInterface>hardware_interface/VelocityJointInterface</hardwareInterface>
+      </joint>
+      <actuator name="${joint}_motor">
+        <hardwareInterface>hardware_interface/VelocityJointInterface</hardwareInterface>
+        <mechanicalReduction>1</mechanicalReduction>
+      </actuator>
+    </transmission>
   </xacro:macro>
   <!--fb : front, back ; lr: left, right -->
@@ -19,12 +32,13 @@
     <link name="${fb}_${lr}_wheel">
       <visual>
-        <origin xyz="0 0 0" rpy="${flipY*pi_2} 0 0 " />
+        <origin xyz="0 0 0" rpy="${flipY*pi_2} 0 ${pi/2.0*(reflect - 1)}" />
         <geometry>
-          <cylinder length="${width}" radius="${radius}" />
+          <!--cylinder length="${width}" radius="${radius}" /-->
+          <mesh filename="package://diffbot_description/meshes/wheel_rim.stl" />
         </geometry>
-        <material name="black" />
+        <material name="yellow" />
       </visual>
       <collision>
-        <origin xyz="0 0 0" rpy="${flipY*pi_2} 0 0 " />
+        <origin xyz="0 0 0" rpy="${flipY*pi_2} 0 0" />
         <geometry>
           <cylinder length="${width}" radius="${radius}" />
@@ -38,10 +52,5 @@
     </link>
     <gazebo reference="${fb}_${lr}_wheel">
-      <mu1 value="200.0"/>
-      <mu2 value="100.0"/>
-      <kp  value="10000000.0" />
-      <kd  value="1.0" />
-      <fdir1 value="1 0 0"/>
-      <material>Gazebo/Grey</material>
+      <material>Gazebo/Yellow</material>
       <turnGravityOff>false</turnGravityOff>
     </gazebo>
@@ -55,14 +64,51 @@
     </joint>
     <!-- Transmission is important to link the joints and the controller -->
-    <transmission name="${fb}_${lr}_wheel_joint_trans">
-      <type>transmission_interface/SimpleTransmission</type>
-      <joint name="${fb}_${lr}_wheel_joint">
-        <hardwareInterface>hardware_interface/VelocityJointInterface</hardwareInterface>
-      </joint>
-      <actuator name="${fb}_${lr}_wheel_joint_motor">
-        <hardwareInterface>hardware_interface/VelocityJointInterface</hardwareInterface>
-        <mechanicalReduction>1</mechanicalReduction>
-      </actuator>
-    </transmission>
+    <xacro:transmission joint="${fb}_${lr}_wheel_joint"/>
+    <!-- Wheel tire - same as wheel tire but without collision and inertia because this is kept in wheel, see above -->
+    <link name="${fb}_${lr}_wheel_tire">
+      <visual>
+        <origin xyz="0 0 0" rpy="${flipY*pi_2} 0 0 " />
+        <geometry>
+          <!--cylinder length="${width}" radius="${radius}" /-->
+          <mesh filename="package://diffbot_description/meshes/wheel_tire.stl" />
+        </geometry>
+        <material name="black" />
+      </visual>
+    </link>
+    <gazebo reference="${fb}_${lr}_wheel_tire">
+      <material>Gazebo/Black</material>
+      <turnGravityOff>false</turnGravityOff>
+    </gazebo>
+    <joint name="${fb}_${lr}_wheel_tire_joint" type="fixed">
+      <parent link="${fb}_${lr}_wheel"/>
+      <child link="${fb}_${lr}_wheel_tire"/>
+      <origin xyz="0 0 0" rpy="0 0 ${pi/2.0*(reflect - 1)}" />
+      <axis xyz="0 1 0" rpy="0 0 0" />
+      <limit effort="100" velocity="100"/>
+      <joint_properties damping="0.0" friction="0.0"/>
+    </joint>
+    <!-- Motor -->
+    <link name="${fb}_${lr}_motor">
+      <visual>
+        <origin xyz="0 0 0" rpy="${flipY*pi} 0 0" />
+        <geometry>
+          <!--cylinder length="${width}" radius="${radius}" /-->
+          <mesh filename="package://diffbot_description/meshes/motor.stl" />
+        </geometry>
+        <material name="blue" />
+      </visual>
+    </link>
+    <joint name="${fb}_${lr}_motor_joint" type="fixed">
+      <parent link="${parent}"/>
+      <child link="${fb}_${lr}_motor"/>
+      <origin xyz="${transX} ${reflect * (transY - wheel_width)} ${transZ}" rpy="${-pi/2.0*(reflect - 1)} 0 0" />
+      <axis xyz="0 1 0" rpy="0 0 ${pi/2.0*(reflect - 1)}" />
+      <limit effort="100" velocity="100"/>
+      <joint_properties damping="0.0" friction="0.0"/>
+    </joint>
+    <gazebo reference="${fb}_${lr}_motor">
+      <material>Gazebo/SkyBlue</material>
+      <turnGravityOff>false</turnGravityOff>
+    </gazebo>
   </xacro:macro>
 </robot>

Commit message: rearrange links and joint tagas

File: ros/src/diffbot_description/urdf/caster_wheel.urdf.xacro (robot description, xacro)
@@ -1,14 +1,7 @@
 <?xml version="1.0"?>
 <robot name="caster_wheel" xmlns:xacro="http://www.ros.org/wiki/xacro">
-    <!--fb : front, back ; lr: left, right -->
+    <!-- caster base (fixed) -->
     <xacro:macro name="caster_wheel" params="locationprefix locationright wheel_base_dx
         flipY:=${1}">
-        <joint name="${locationprefix}_caster_base_joint" type="fixed">
-            <origin xyz="${wheel_base_dx} ${-caster_wheel_base_dy * locationright} ${caster_wheel_base_dz}" rpy="0 0 0" />
-            <parent link="base_link" />
-            <child link="${locationprefix}_caster_base_link" />
-            <axis xyz="0 0 1" />
-            <dynamics damping="0.01" friction="0.0"/>
-        </joint>
         <link name="${locationprefix}_caster_base_link">
             <inertial>
@@ -33,15 +26,15 @@
             </collision>
         </link>
+        <joint name="${locationprefix}_caster_base_joint" type="fixed">
+            <origin xyz="${wheel_base_dx} ${-caster_wheel_base_dy * locationright} ${caster_wheel_base_dz}" rpy="0 0 0" />
+            <parent link="base_link" />
+            <child link="${locationprefix}_caster_base_link" />
+            <axis xyz="0 0 1" />
+            <dynamics damping="0.01" friction="0.0"/>
+        </joint>
         <gazebo reference="${locationprefix}_caster_base_link">
             <material>Gazebo/Grey</material>
         </gazebo>
         <!-- caster hub -->
-        <joint name="${locationprefix}_caster_rotation_joint" type="continuous">
-            <origin xyz="${wheel_base_dx} ${-caster_wheel_base_dy * locationright} ${caster_wheel_base_dz}" rpy="0 0 0" />
-            <parent link="base_link" />
-            <child link="${locationprefix}_caster_rotation_link" />
-            <axis xyz="0 0 1" />
-            <dynamics damping="0.01" friction="0.0"/>
-        </joint>
         <link name="${locationprefix}_caster_rotation_link">
             <inertial>
@@ -66,14 +59,15 @@
             </collision>
         </link>
+        <joint name="${locationprefix}_caster_rotation_joint" type="continuous">
+            <origin xyz="${wheel_base_dx} ${-caster_wheel_base_dy * locationright} ${caster_wheel_base_dz}" rpy="0 0 0" />
+            <parent link="base_link" />
+            <child link="${locationprefix}_caster_rotation_link" />
+            <axis xyz="0 0 1" />
+            <dynamics damping="0.01" friction="0.0"/>
+        </joint>
         <gazebo reference="${locationprefix}_caster_rotation_link">
             <material>Gazebo/Grey</material>
         </gazebo>
         <!-- caster wheel -->
-        <joint name="${locationprefix}_caster_wheel_joint" type="continuous">
-            <origin xyz="${caster_wheel_dx} ${-caster_wheel_dy * locationright} ${caster_wheel_dz}" rpy="0 0 0" />
-            <parent link="${locationprefix}_caster_rotation_link" />
-            <child link="${locationprefix}_caster_wheel_link" />
-            <axis xyz="0 1 0" />
-        </joint>
         <link name="${locationprefix}_caster_wheel_link">
             <xacro:cylinder_inertial mass="${caster_wheel_mass}" radius="${caster_wheel_radius}" length="${caster_wheel_width}">
@@ -96,4 +90,10 @@
             </collision>
         </link>
+        <joint name="${locationprefix}_caster_wheel_joint" type="continuous">
+            <origin xyz="${caster_wheel_dx} ${-caster_wheel_dy * locationright} ${caster_wheel_dz}" rpy="0 0 0" />
+            <parent link="${locationprefix}_caster_rotation_link" />
+            <child link="${locationprefix}_caster_wheel_link" />
+            <axis xyz="0 1 0" />
+        </joint>
         <gazebo reference="${locationprefix}_caster_wheel_link">
             <material>Gazebo/DarkGrey</material>
