Commit message: add diffbot description files xacro and gazebo

File: ros/src/diffbot_description/urdf/diffbot.xacro (robot description, xacro)
@@ -1,38 +1,16 @@
 <?xml version="1.0"?>
 <robot name="diffbot" xmlns:xacro="http://ros.org/wiki/xacro">
-  <xacro:include filename="$(find diffbot_description)/urdf/wheel.urdf.xacro" />
-  <!-- Defining the colors used in this robot -->
-  <material name="black">
-    <color rgba="0.0 0.0 0.0 1.0"/>
-  </material>
-  <material name="red">
-    <color rgba="0.8 0.0 0.0 1.0"/>
-  </material>
-  <material name="yellow">
-    <color rgba="0.9 0.7 0.1 1.0"/>
-  </material>
-  <material name="white">
-    <color rgba="1.0 1.0 1.0 1.0"/>
-  </material>
-  <material name="blue">
-    <color rgba="0.0 0.0 0.8 1.0"/>
-  </material>
-  <!-- PROPERTY LIST -->
+  <!-- Properties -->
   <!--All units in m-kg-s-radians unit system -->
+  <!-- Constants for robot dimensions -->
   <xacro:property name="M_PI" value="3.1415926535897931" />
   <xacro:property name="M_PI_2" value="1.570796327" />
   <xacro:property name="DEG_TO_RAD" value="0.017453293" />
-  <!-- Main body width, length and height -->
-  <!-- Main body box base   -->
+  <!-- Main body height, length width and mass -->
+  <!-- Main body box base -->
   <xacro:property name="base_height" value="0.02" />
   <xacro:property name="base_length" value="0.30" />
   <xacro:property name="base_width" value="0.15" />
   <xacro:property name="base_mass" value="5" /> <!-- in kg-->
-  <!-- Macro for box geometry -->
-  <xacro:macro name="box_geometry" params="length:=${base_length} width:=${base_width} ${base_height}">
-    <geometry>
-      <box size="${length} ${width} ${height}" />
-    </geometry>
-  </xacro:macro>
   <!-- Macro for calculating inertia of box, see https://en.wikipedia.org/wiki/List_of_moments_of_inertia -->
   <xacro:macro name="box_inertia" params="m w h d">
@@ -41,13 +19,14 @@
               izz="${m/12*(w*w + h*h)}" />
   </xacro:macro>
-  <!-- Wheels -->
+  <!-- Wheel properties -->
+  <!-- Wheel radius, width and mass -->
   <xacro:property name="wheel_radius" value="0.04" />
   <xacro:property name="wheel_width" value="0.02" />
   <xacro:property name="wheel_mass" value="2.5" /> <!-- in kg-->
+  <!-- Wheel placement relative to base origin -->
   <xacro:property name="base_x_origin_to_wheel_origin" value="${base_length/2.0*0.7}" />
   <xacro:property name="base_y_origin_to_wheel_origin" value="${base_width/2.0}" />
   <xacro:property name="base_z_origin_to_wheel_origin" value="0.0" />
-  <!-- Caster wheel radius and height -->
-  <!-- Caster wheel mass -->
+  <!-- Caster wheel radius, width and mass -->
   <xacro:property name="caster_height" value="0.04" />
   <xacro:property name="caster_radius" value="0.025" />
@@ -55,5 +34,10 @@
   <!-- Hokuyo Laser scanner -->
   <xacro:property name="hokuyo_size" value="0.05" />
-  <!-- BASE-FOOTPRINT -->
+  <xacro:include filename="$(find diffbot_description)/urdf/wheel.urdf.xacro" />
+  <!-- Import all Gazebo-customization elements, including Gazebo colors -->
+  <xacro:include filename="$(find diffbot_description)/urdf/diffbot.gazebo" />
+  <!-- Import RViz colors -->
+  <xacro:include filename="$(find diffbot_description)/urdf/materials.xacro" />
+  <!-- Base-Footprint -->
   <!-- base_footprint is a fictitious link(frame) that is on the ground right below base_link origin -->
   <link name="base_footprint">
@@ -65,7 +49,5 @@
     </collision>
   </link>
-  <gazebo reference="base_footprint">
-    <turnGravityOff>false</turnGravityOff>
-  </gazebo>
+  <!-- Joint to connect base_footprint with base_link -->
   <joint name="base_footprint_joint" type="fixed">
     <origin xyz="0 0 ${wheel_radius - base_z_origin_to_wheel_origin}" rpy="0 0 0" />
@@ -73,6 +55,6 @@
     <child link="base_link" />
   </joint>
-  <!-- BASE-LINK -->
-  <!--Actual body/chassis of the robot-->
+  <!-- Base-Link -->
+  <!-- Actual body/chassis of the robot-->
   <link name="base_link">
     <inertial>
@@ -96,8 +78,10 @@
     </collision>
   </link>
-  <gazebo reference="base_link">
-    <material>Gazebo/White</material>
-    <turnGravityOff>false</turnGravityOff>
-  </gazebo>
+  <!-- Joint between base_link and back caster wheel -->
+  <joint name="caster_joint" type="fixed">
+    <parent link="base_link"/>
+    <child link="caster_link"/>
+    <origin xyz="-0.135 0.0 0.009" rpy="${-M_PI/2} 0 0"/>
+  </joint>
   <!-- Caster back  -->
   <link name="caster_link">
@@ -123,13 +107,5 @@
       </inertial>
   </link>
-  <joint name="caster_joint" type="fixed">
-    <parent link="base_link"/>
-    <child link="caster_link"/>
-    <origin xyz="-0.135 0.0 0.009" rpy="${-M_PI/2} 0 0"/>
-  </joint>
-  <gazebo reference="caster_link">
-    <turnGravityOff>false</turnGravityOff>
-  </gazebo>
-  <!-- Wheel Definitions -->
+  <!-- Wheel definitions -->
   <xacro:wheel fb="front" lr="right" parent="base_link"
     mass="${wheel_mass}" radius="${wheel_radius}" width="${wheel_width}" reflect="1"
@@ -144,27 +120,3 @@
     transZ="${base_z_origin_to_wheel_origin}"
     flipY="1" />
-  <!-- Differential drive controller  -->
-  <gazebo>
-    <plugin name="differential_drive_controller" filename="libgazebo_ros_diff_drive.so">
-      <legacyMode>true</legacyMode>
-      <rosDebugLevel>Debug</rosDebugLevel>
-      <publishWheelTF>false</publishWheelTF>
-      <robotNamespace>/</robotNamespace>
-      <publishTf>1</publishTf>
-      <publishWheelJointState>false</publishWheelJointState>
-      <alwaysOn>true</alwaysOn>
-      <updateRate>100.0</updateRate>
-      <leftJoint>front_left_wheel_joint</leftJoint>
-      <rightJoint>front_right_wheel_joint</rightJoint>
-      <wheelSeparation>${2*base_width}</wheelSeparation>
-      <wheelDiameter>${2*wheel_radius}</wheelDiameter>
-      <broadcastTF>1</broadcastTF>
-      <wheelTorque>30</wheelTorque>
-      <wheelAcceleration>1.8</wheelAcceleration>
-      <commandTopic>cmd_vel</commandTopic>
-      <odometryFrame>odom</odometryFrame>
-      <odometryTopic>odom</odometryTopic>
-      <robotBaseFrame>base_footprint</robotBaseFrame>
-    </plugin>
-  </gazebo>
 </robot>

Commit message: update diffbot_description

File: ros/src/diffbot_description/urdf/diffbot.xacro (robot description, xacro)
@@ -23,5 +23,5 @@
   <xacro:property name="wheel_radius" value="0.04" />
   <xacro:property name="wheel_width" value="0.02" />
-  <xacro:property name="wheel_mass" value="2.5" /> <!-- in kg-->
+  <xacro:property name="wheel_mass" value="0.1" /> <!-- in kg-->
   <!-- Wheel placement relative to base origin -->
   <xacro:property name="base_x_origin_to_wheel_origin" value="${base_length/2.0*0.7}" />

Commit message: change inertial matrices and masses

File: ros/src/diffbot_description/urdf/diffbot.xacro (robot description, xacro)
@@ -12,10 +12,15 @@
   <xacro:property name="base_length" value="0.30" />
   <xacro:property name="base_width" value="0.15" />
-  <xacro:property name="base_mass" value="5" /> <!-- in kg-->
+  <xacro:property name="base_mass" value="16.0" /> <!-- in kg-->
   <!-- Macro for calculating inertia of box, see https://en.wikipedia.org/wiki/List_of_moments_of_inertia -->
-  <xacro:macro name="box_inertia" params="m w h d">
-    <inertia  ixx="${m/12*(h*h + d*d)}" ixy = "0" ixz = "0"
-              iyy="${m/12*(w*w + d*d)}" iyz = "0"
-              izz="${m/12*(w*w + h*h)}" />
+  <xacro:macro name="box_inertia" params="m l w h">
+    <inertia  ixx="${m/12*(w*w + h*h)}" ixy = "0" ixz = "0"
+              iyy="${m/12*(l*l + h*h)}" iyz = "0"
+              izz="${m/12*(l*l + w*w)}" />
+  </xacro:macro>
+  <xacro:macro name="sphere_inertia" params="m r">
+    <inertia  ixx="${m*2/5*r*r}" ixy = "0" ixz = "0"
+              iyy="${m*2/5*r*r}" iyz = "0"
+              izz="${m*2/5*r*r}" />
   </xacro:macro>
   <!-- Wheel properties -->
@@ -23,5 +28,5 @@
   <xacro:property name="wheel_radius" value="0.04" />
   <xacro:property name="wheel_width" value="0.02" />
-  <xacro:property name="wheel_mass" value="0.1" /> <!-- in kg-->
+  <xacro:property name="wheel_mass" value="1.0" /> <!-- in kg-->
   <!-- Wheel placement relative to base origin -->
   <xacro:property name="base_x_origin_to_wheel_origin" value="${base_length/2.0*0.7}" />
@@ -31,5 +36,5 @@
   <xacro:property name="caster_height" value="0.04" />
   <xacro:property name="caster_radius" value="0.025" />
-  <xacro:property name="caster_mass" value="0.5" /> <!-- in kg-->
+  <xacro:property name="caster_mass" value="1.0" /> <!-- in kg-->
   <!-- Hokuyo Laser scanner -->
   <xacro:property name="hokuyo_size" value="0.05" />
@@ -61,6 +66,6 @@
       <mass value="${base_mass}" />
       <origin xyz="0 0 0" />
-        <!--The 3x3 rotational inertia matrix. -->
-        <xacro:box_inertia  m="${base_mass}" w="${base_width}" h="${base_length}" d="${base_height}" />
+      <!--The 3x3 rotational inertia matrix. -->
+      <xacro:box_inertia  m="${base_mass}" l="${base_length}" w="${base_width}" h="${base_height}" />
     </inertial>
     <visual>
@@ -72,5 +77,5 @@
     </visual>
     <collision>
-      <origin xyz="0 0 0" rpy="0 0 0 " />
+      <origin xyz="0 0 0" rpy="0 0 0" />
       <geometry>
           <box size="${base_length} ${base_width} ${base_height}" />
@@ -82,10 +87,10 @@
     <parent link="base_link"/>
     <child link="caster_link"/>
-    <origin xyz="-0.135 0.0 0.009" rpy="${-M_PI/2} 0 0"/>
+    <origin xyz="-0.12 0.0 -0.02" rpy="0 0 0"/>
   </joint>
   <!-- Caster back  -->
   <link name="caster_link">
     <visual>
-      <origin xyz="0.02 0.02 0 " rpy="${M_PI/2} 0 0" />
+      <origin xyz="0 0 0" rpy="0 0 0" />
       <geometry>
         <sphere radius="${caster_radius}" />
@@ -94,17 +99,25 @@
     </visual>
     <collision>
+      <origin xyz="0 0 0" rpy="0 0 0" />
       <geometry>
         <sphere radius="${caster_radius}" />
       </geometry>
-      <origin xyz="0 0.02 0 " rpy="${M_PI/2} 0 0" />
     </collision>
     <inertial>
       <mass value="${caster_mass}" />
       <origin xyz="0 0 0" />
-      <inertia ixx="0.001" ixy="0.0" ixz="0.0"
-               iyy="0.001" iyz="0.0"
-               izz="0.001" />
-      </inertial>
+      <!--The 3x3 rotational inertia matrix. -->
+      <xacro:sphere_inertia  m="${caster_mass}" r="${caster_radius}" />
+    </inertial>
   </link>
+  <!--gazebo reference="caster_link">
+      <mu1 value="1.0"/>
+      <mu2 value="1.0"/>
+      <kp  value="10000000.0" />
+      <kd  value="1.0" />
+      <fdir1 value="1 0 0"/>
+      <material>Gazebo/Grey</material>
+      <turnGravityOff>false</turnGravityOff>
+    </gazebo-->
   <!-- Wheel definitions -->
   <xacro:wheel fb="front" lr="right" parent="base_link"

Commit message: use new xacro macro caster wheel and other includes

File: ros/src/diffbot_description/urdf/diffbot.xacro (robot description, xacro)
@@ -4,7 +4,7 @@
   <!--All units in m-kg-s-radians unit system -->
   <!-- Constants for robot dimensions -->
-  <xacro:property name="M_PI" value="3.1415926535897931" />
-  <xacro:property name="M_PI_2" value="1.570796327" />
-  <xacro:property name="DEG_TO_RAD" value="0.017453293" />
+  <!--xacro:property name="pi" value="3.1415926535897931" /-->
+  <xacro:property name="pi_2" value="1.570796327" />
+  <xacro:property name="deg_to_rad" value="0.017453293" />
   <!-- Main body height, length width and mass -->
   <!-- Main body box base -->
@@ -34,12 +34,24 @@
   <xacro:property name="base_z_origin_to_wheel_origin" value="0.0" />
   <!-- Caster wheel radius, width and mass -->
-  <xacro:property name="caster_height" value="0.04" />
-  <xacro:property name="caster_radius" value="0.025" />
-  <xacro:property name="caster_mass" value="1.0" /> <!-- in kg-->
+  <xacro:property name="caster_wheel_width" value="0.01" />
+  <xacro:property name="caster_wheel_radius" value="0.015" />
+  <xacro:property name="caster_wheel_mass" value="1.0" /> <!-- in kg-->
+  <!-- Caster wheel base size, width and mass -->
+  <xacro:property name="caster_wheel_dx" value="${-caster_base_size/2.0}" />
+  <xacro:property name="caster_wheel_dy" value="-1" />
+  <xacro:property name="caster_wheel_dz" value="${-caster_base_size}" />
+  <!--xacro:property name="front_caster_wheel_base_dx" value="0.341346" /-->
+  <xacro:property name="caster_base_size" value="0.02" />
+  <xacro:property name="back_caster_wheel_base_dx" value="-0.270154" />
+  <xacro:property name="caster_wheel_base_dy" value="0.203" />
+  <xacro:property name="caster_wheel_base_dz" value="${-base_height/2.0}" />
   <!-- Hokuyo Laser scanner -->
   <xacro:property name="hokuyo_size" value="0.05" />
+  <!-- Import all Gazebo-customization elements, including Gazebo colors -->
+  <xacro:include filename="$(find diffbot_description)/urdf/common_properties.urdf.xacro" />
   <xacro:include filename="$(find diffbot_description)/urdf/wheel.urdf.xacro" />
-  <!-- Import all Gazebo-customization elements, including Gazebo colors -->
-  <xacro:include filename="$(find diffbot_description)/urdf/diffbot.gazebo" />
+  <xacro:include filename="$(find diffbot_description)/urdf/caster_wheel.urdf.xacro" />
+  <xacro:include filename="$(find diffbot_description)/urdf/diffbot_colors.gazebo.xacro" />
+  <xacro:include filename="$(find diffbot_description)/urdf/diffbot.gazebo.xacro" />
   <!-- Import RViz colors -->
   <xacro:include filename="$(find diffbot_description)/urdf/materials.xacro" />
@@ -83,41 +95,4 @@
     </collision>
   </link>
-  <!-- Joint between base_link and back caster wheel -->
-  <joint name="caster_joint" type="fixed">
-    <parent link="base_link"/>
-    <child link="caster_link"/>
-    <origin xyz="-0.12 0.0 -0.02" rpy="0 0 0"/>
-  </joint>
-  <!-- Caster back  -->
-  <link name="caster_link">
-    <visual>
-      <origin xyz="0 0 0" rpy="0 0 0" />
-      <geometry>
-        <sphere radius="${caster_radius}" />
-      </geometry>
-      <material name="black" />
-    </visual>
-    <collision>
-      <origin xyz="0 0 0" rpy="0 0 0" />
-      <geometry>
-        <sphere radius="${caster_radius}" />
-      </geometry>
-    </collision>
-    <inertial>
-      <mass value="${caster_mass}" />
-      <origin xyz="0 0 0" />
-      <!--The 3x3 rotational inertia matrix. -->
-      <xacro:sphere_inertia  m="${caster_mass}" r="${caster_radius}" />
-    </inertial>
-  </link>
-  <!--gazebo reference="caster_link">
-      <mu1 value="50.0"/>
-      <mu2 value="25.0"/>
-      <kp  value="10000.0" />
-      <kd  value="1.0" />
-      <fdir1 value="1 0 0"/>
-      <material>Gazebo/Grey</material>
-      <turnGravityOff>false</turnGravityOff>
-    </gazebo-->
   <!-- Wheel definitions -->
   <xacro:wheel fb="front" lr="right" parent="base_link"
@@ -133,3 +108,6 @@
     transZ="${base_z_origin_to_wheel_origin}"
     flipY="1" />
+    <!-- Caster back  -->
+    <!-- Joint between base_link and back caster wheel -->
+    <xacro:caster_wheel locationprefix="back" locationright="0" wheel_base_dx="${-base_length/2.0*0.9}" />
 </robot>

Commit message: move macros to common_properties and fix masses of caster

File: ros/src/diffbot_description/urdf/diffbot.xacro (robot description, xacro)
@@ -13,15 +13,4 @@
   <xacro:property name="base_width" value="0.15" />
   <xacro:property name="base_mass" value="16.0" /> <!-- in kg-->
-  <!-- Macro for calculating inertia of box, see https://en.wikipedia.org/wiki/List_of_moments_of_inertia -->
-  <xacro:macro name="box_inertia" params="m l w h">
-    <inertia  ixx="${m/12*(w*w + h*h)}" ixy = "0" ixz = "0"
-              iyy="${m/12*(l*l + h*h)}" iyz = "0"
-              izz="${m/12*(l*l + w*w)}" />
-  </xacro:macro>
-  <xacro:macro name="sphere_inertia" params="m r">
-    <inertia  ixx="${m*2/5*r*r}" ixy = "0" ixz = "0"
-              iyy="${m*2/5*r*r}" iyz = "0"
-              izz="${m*2/5*r*r}" />
-  </xacro:macro>
   <!-- Wheel properties -->
   <!-- Wheel radius, width and mass -->
@@ -36,5 +25,5 @@
   <xacro:property name="caster_wheel_width" value="0.01" />
   <xacro:property name="caster_wheel_radius" value="0.015" />
-  <xacro:property name="caster_wheel_mass" value="1.0" /> <!-- in kg-->
+  <xacro:property name="caster_wheel_mass" value="0.5" /> <!-- in kg-->
   <!-- Caster wheel base size, width and mass -->
   <xacro:property name="caster_wheel_dx" value="${-caster_base_size/2.0}" />
@@ -42,4 +31,5 @@
   <xacro:property name="caster_wheel_dz" value="${-caster_base_size}" />
   <!--xacro:property name="front_caster_wheel_base_dx" value="0.341346" /-->
+  <xacro:property name="caster_base_mass" value="0.02" />
   <xacro:property name="caster_base_size" value="0.02" />
   <xacro:property name="back_caster_wheel_base_dx" value="-0.270154" />

Commit message: add camera to diffbot robot description

File: ros/src/diffbot_description/urdf/diffbot.xacro (robot description, xacro)
@@ -35,6 +35,12 @@
   <xacro:property name="caster_wheel_base_dy" value="0.203" />
   <xacro:property name="caster_wheel_base_dz" value="0.002" />
-  <!-- Hokuyo Laser scanner -->
-  <xacro:property name="hokuyo_size" value="0.05" />
+  <!-- Sensors -->
+  <!-- Camera -->
+  <xacro:property name="camera_size" value="0.02" /> <!-- Size of square 'camera' box -->
+  <xacro:property name="camera_dx" value="${base_length/2.0*0.8}" />
+  <xacro:property name="camera_dy" value="0.0" />
+  <xacro:property name="camera_dz" value="${camera_size/2.0}" />
+  <!-- Laser scanner -->
+  <xacro:property name="lidar_size" value="0.05" />
   <!-- Import all Gazebo-customization elements, including Gazebo colors -->
   <xacro:include filename="$(find diffbot_description)/urdf/common_properties.urdf.xacro" />
@@ -43,4 +49,5 @@
   <xacro:include filename="$(find diffbot_description)/urdf/diffbot_colors.gazebo.xacro" />
   <xacro:include filename="$(find diffbot_description)/urdf/diffbot.gazebo.xacro" />
+  <xacro:include filename="$(find diffbot_description)/urdf/sensors.gazebo.xacro" />
   <!-- Import RViz colors -->
   <xacro:include filename="$(find diffbot_description)/urdf/materials.xacro" />

File: ros/src/diffbot_description/urdf/diffbot_colors.gazebo.xacro (robot description, xacro)
@@ -14,76 +14,3 @@
     <turnGravityOff>false</turnGravityOff>
   </gazebo>
-  <!-- Differential drive controller -->
-  <!--
-  <gazebo>
-    <plugin name="differential_drive_controller" filename="libgazebo_ros_diff_drive.so">
-      <legacyMode>true</legacyMode>
-      <rosDebugLevel>Debug</rosDebugLevel>
-      <publishWheelTF>false</publishWheelTF>
-      <robotNamespace>/</robotNamespace>
-      <publishTf>1</publishTf>
-      <publishWheelJointState>false</publishWheelJointState>
-      <alwaysOn>true</alwaysOn>
-      <updateRate>100.0</updateRate>
-      <leftJoint>front_left_wheel_joint</leftJoint>
-      <rightJoint>front_right_wheel_joint</rightJoint>
-      <wheelSeparation>${2*base_width}</wheelSeparation>
-      <wheelDiameter>${2*wheel_radius}</wheelDiameter>
-      <broadcastTF>1</broadcastTF>
-      <wheelTorque>30</wheelTorque>
-      <wheelAcceleration>1.8</wheelAcceleration>
-      <commandTopic>cmd_vel</commandTopic>
-      <odometryFrame>odom</odometryFrame>
-      <odometryTopic>odom</odometryTopic>
-      <robotBaseFrame>base_footprint</robotBaseFrame>
-    </plugin>
-  </gazebo>
-  -->
-  <!-- camera -->
-  <gazebo reference="camera_link">
-    <sensor type="camera" name="camera1">
-      <update_rate>30.0</update_rate>
-      <camera name="head">
-        <horizontal_fov>1.3962634</horizontal_fov>
-        <image>
-          <width>800</width>
-          <height>800</height>
-          <format>R8G8B8</format>
-        </image>
-        <clip>
-          <near>0.02</near>
-          <far>300</far>
-        </clip>
-        <noise>
-          <type>gaussian</type>
-          <!-- Noise is sampled independently per pixel on each frame.
-               That pixel's noise value is added to each of its color
-               channels, which at that point lie in the range [0,1]. -->
-          <mean>0.0</mean>
-          <stddev>0.007</stddev>
-        </noise>
-      </camera>
-      <plugin name="camera_controller" filename="libgazebo_ros_camera.so">
-        <alwaysOn>true</alwaysOn>
-        <updateRate>0.0</updateRate>
-        <cameraName>rrbot/camera1</cameraName>
-        <imageTopicName>image_raw</imageTopicName>
-        <cameraInfoTopicName>camera_info</cameraInfoTopicName>
-        <frameName>camera_link_optical</frameName>
-        <!-- setting hackBaseline to anything but 0.0 will cause a misalignment
-            between the gazebo sensor image and the frame it is supposed to
-            be attached to -->
-        <hackBaseline>0.0</hackBaseline>
-        <distortionK1>0.0</distortionK1>
-        <distortionK2>0.0</distortionK2>
-        <distortionK3>0.0</distortionK3>
-        <distortionT1>0.0</distortionT1>
-        <distortionT2>0.0</distortionT2>
-        <CxPrime>0</CxPrime>
-        <Cx>0.0</Cx>
-        <Cy>0.0</Cy>
-        <focalLength>0.0</focalLength>
-      </plugin>
-    </sensor>
-  </gazebo>
 </robot>

File: ros/src/diffbot_description/urdf/materials.xacro (robot description, xacro)
@@ -17,3 +17,6 @@
     <color rgba="0.0 0.0 0.8 1.0"/>
   </material>
+  <material name="green">
+    <color rgba="0.04 0.4 0.14 1.0"/>
+  </material>
 </robot>
