Commit message: add colors for gazebo

File: diffbot_description/urdf/include/common_macros.urdf.xacro (robot description, xacro)
@@ -54,4 +54,7 @@
       </xacro:cylinder_inertia>
     </link>
+    <gazebo reference="${prefix}_wheel">
+      <material>Gazebo/Grey</material>
+    </gazebo>
     <joint name="${prefix}_wheel_joint" type="continuous">
       <axis xyz="0 1 0" rpy="0 0 0" />
@@ -267,8 +270,8 @@
       <!--axis xyz="0 1 0" rpy="0 0 ${pi/2.0*(reflect - 1)}" /-->
     </joint>
-    <!--gazebo reference="${fb}_${lr}_motor">
+    <gazebo reference="${prefix}_motor">
       <material>Gazebo/SkyBlue</material>
       <turnGravityOff>false</turnGravityOff>
-    </gazebo-->
+    </gazebo>
   </xacro:macro>
 <!-- ===================== Base xacro ==========================================

File: diffbot_description/urdf/include/common_sensors.xacro (robot description, xacro)
@@ -36,4 +36,7 @@
       </xacro:cylinder_inertia>
   </link>
+  <gazebo reference="${prefix}_gpu_laser_link">
+    <material>Gazebo/Grey</material>
+  </gazebo>
   <joint name="${prefix}_gpu_laser_joint" type="fixed">
     <parent link="${parent_link}"/>

Commit message: add z_offset to diffbot base_footprint description for moving on the ground in rviz

File: diffbot_description/urdf/include/common_macros.urdf.xacro (robot description, xacro)
@@ -339,5 +339,5 @@
       <!-- origin xyz="0 0 ${wheel_radius - base_z_origin_to_wheel_origin}" rpy="0 0 0" /-->
       <!-- origin xyz="0 0 ${wheel_props['wheel']['radius'] - wheel_props['wheel']['z_offset'] + 0.1}" rpy="0 0 0" /-->
-      <origin xyz="0 0 0" rpy="0 0 0" />
+      <origin xyz="0 0 ${wheel_props['wheel']['radius'] - wheel_props['wheel']['z_offset']}" rpy="0 0 0" />
     </joint>
   </xacro:macro>
