Commit message: DiffBot: sphere collision for the drive wheels, so they touch the ground in their center plane
In Gazebo, DiffBot turned 16 % less on the spot than its wheels and its odometry said, while its
wheels followed their commands. The ratio matched an effective wheel separation between the
wheels' outer edges, 0.160 m instead of 0.135 m: with the default contact settings, Gazebo put
the contacts of DiffBot's collision cylinders at their outer edges. At 1.0 rad/s, the robot
turned 2.53 rad for 3.0 commanded (0.135 / 0.160 = 0.844); with 5 mm wide collision cylinders,
3.37 rad (0.135 / 0.120 = 1.125). A sphere with the wheel's radius touches the ground at one
point in the wheel's center plane: DiffBot then turns 2.99 rad. The visual stays a cylinder.

Part of #118

File: diffbot_description/urdf/include/common_macros.urdf.xacro (robot description, xacro)
@@ -46,8 +46,12 @@
       </visual>
     </xacro:if>
+      <!-- A sphere with the wheel's radius, so the wheel touches the ground at one point in its
+           center plane. With the cylinder, Gazebo put DiffBot's contacts at the wheels' outer
+           edges, which made the wheel separation 0.160 m instead of 0.135 m: the robot turned 16 %
+           less than its wheels and its odometry (ros-mobile-robots/diffbot#118). The visual
+           stays a cylinder -->
       <collision>
-        <origin xyz="0 0 0" rpy="${pi/2} 0 0"/>
-        <geometry>
-          <cylinder radius="${wheel_props['radius']}" length="${wheel_props['length']}"/>
+        <geometry>
+          <sphere radius="${wheel_props['radius']}"/>
         </geometry>
       </collision>

Commit message: DiffBot: sphere collision for the drive wheels, so they touch the ground in their center plane (#120)
In Gazebo, DiffBot's collision cylinders touched the ground at their outer edges, so it turned about 15 % less than its odometry: 0.138 / 0.163 m, its wheel separation over the distance between the outer edges. A sphere with the wheel radius touches the ground at one point in the wheel's center plane. The visual (mesh) and the cylinder inertia are unchanged. test_drive.py's comments have the new values; no check changed.

Part of #118

File: diffbot_description/urdf/include/common_macros.urdf.xacro (robot description, xacro)
@@ -46,8 +46,12 @@
       </visual>
     </xacro:if>
+      <!-- Use a sphere with the wheel radius for collision. On flat ground, an upright wheel's
+           contact stays in its center plane. This avoids the outer-edge cylinder contacts that
+           can increase DiffBot's effective wheel separation and reduce its true turn relative
+           to odometry. The wheel visual and cylinder inertia are unchanged.
+           See https://github.com/ros-mobile-robots/diffbot/pull/120 -->
       <collision>
-        <origin xyz="0 0 0" rpy="${pi/2} 0 0"/>
-        <geometry>
-          <cylinder radius="${wheel_props['radius']}" length="${wheel_props['length']}"/>
+        <geometry>
+          <sphere radius="${wheel_props['radius']}"/>
         </geometry>
       </collision>
