Commit message: red_w

File: diffbot_description/urdf/include/addon_macro.urdf.xacro (robot description, xacro)
@@ -23,5 +23,5 @@
           <mesh filename="package://${package_name}/meshes/${robot_name}/${base_prop[addon]['mesh']}" scale="${base_prop[addon]['scale']}"/>
         </geometry>
-        <material name="white" />
+        <material name="red" />
       </visual>
     </xacro:if>
