Commit message: include gpu_laser - rplidar a2 for diffbot

File: diffbot_description/urdf/diffbot.urdf.xacro (robot description, xacro)
@@ -14,4 +14,6 @@
   <xacro:property name="base_yaml" value="$(find ${package_name})/config/${robot_name}/base.yaml" />
   <xacro:property name="base_props" value="${load_yaml(base_yaml)}"/>
+  <xacro:property name="sensor_yaml" value="$(find ${package_name})/config/${robot_name}/sensors.yaml" />
+  <xacro:property name="sensor_prop" value="${load_yaml(sensor_yaml)}"/>
   <!-- Footprint link -->
   <xacro:footprint wheel_props="${front_wheel_props}" />
@@ -47,3 +49,6 @@
   </xacro:motor>
   <!-- Sensors -->
+  <xacro:gpu_laser prefix="rplidar" parent_link="base_link"
+                   sensor_prop="${sensor_prop}">
+  </xacro:gpu_laser>
 </robot>

File: diffbot_description/urdf/include/common_sensors.xacro (robot description, xacro)
@@ -1,35 +1,50 @@
 <?xml version="1.0"?>
 <robot xmlns:xacro="http://www.ros.org/wiki/xacro">
-<xacro:macro name="hokuyo_sensor" params=" *joint_origin parent_link ">
-  <link name="hokuyo_link">
-      <collision>
-         <origin xyz="0 0 0" rpy="0 0 0"/>
-        <geometry>
-          <box size="0.06 0.06 0.087"/>
-        </geometry>
-      </collision>
+<xacro:macro name="gpu_laser" params="prefix parent_link sensor_prop ">
+  <xacro:property name="mesh"
+     value="${sensor_prop['gpu_laser']['mesh']}"/>
+  <link name="${prefix}_gpu_laser_link">
+      <xacro:if value="${mesh != '' }" >
       <visual>
         <origin xyz="0 0 0" rpy="0 0 0"/>
         <geometry>
-          <mesh filename="package://${package_name}/meshes/sensors/hokuyo.dae" />
+          <mesh filename="package://${package_name}/meshes/sensors/${mesh}" />
         </geometry>
+        <material name="dark_grey"/>
       </visual>
-      <inertial>
-        <mass value="1e-5" />
+    </xacro:if>
+    <xacro:if value="${mesh == '' }" >
+      <visual>
         <origin xyz="0 0 0" rpy="0 0 0"/>
-        <inertia ixx="1e-6" ixy="0" ixz="0" iyy="1e-6" iyz="0" izz="1e-6" />
-      </inertial>
+         <geometry>
+         <cylinder radius="${sensor_prop['gpu_laser']['radius']}" length="${sensor_prop['gpu_laser']['length']}"/>
+        </geometry>
+        <material name="red"/>
+      </visual>
+    </xacro:if>
+      <collision>
+        <origin xyz="0 0 0" rpy="0 0 0"/>
+        <geometry>
+          <cylinder radius="${sensor_prop['gpu_laser']['radius']}" length="${sensor_prop['gpu_laser']['length']}"/>
+        </geometry>
+      </collision>
+      <xacro:cylinder_inertia m="${sensor_prop['gpu_laser']['mass']}"
+                              r="${sensor_prop['gpu_laser']['radius']}"
+                              l="${sensor_prop['gpu_laser']['length']}"
+                              o_xyz="0 0 0"
+                              o_rpy="0 0 0" >
+      </xacro:cylinder_inertia>
   </link>
-  <joint name="hokuyo_joint" type="fixed">
+  <joint name="${prefix}_gpu_laser_joint" type="fixed">
+    <parent link="${parent_link}"/>
+    <child link="${prefix}_gpu_laser_link"/>
+    <origin xyz="${sensor_prop['gpu_laser']['dx']} ${sensor_prop['gpu_laser']['dy']} ${sensor_prop['gpu_laser']['dz']}" rpy="0 0 0"/>
     <axis xyz="0 1 0" />
-    <xacro:insert_block name="joint_origin" />
-    <parent link="${parent_link}"/>
-    <child link="hokuyo_link"/>
   </joint>
   <!-- hokuyo gazebo references -->
-  <gazebo reference="hokuyo_link">
+  <gazebo reference="${prefix}_gpu_laser_link">
     <sensor type="gpu_ray" name="head_hokuyo_sensor">
       <pose>0 0 0 0 0 0</pose>
-      <visualize>false</visualize>
+      <visualize>true</visualize>
       <update_rate>40</update_rate>
       <ray>
@@ -38,6 +53,6 @@
             <samples>720</samples>
             <resolution>1</resolution>
-            <min_angle>-1.570796</min_angle>
-            <max_angle>1.570796</max_angle>
+            <min_angle>${sensor_prop['gpu_laser']['angular_range']['min']}</min_angle>
+            <max_angle>${sensor_prop['gpu_laser']['angular_range']['max']}</max_angle>
           </horizontal>
         </scan>
@@ -59,5 +74,5 @@
       <plugin name="gazebo_ros_head_hokuyo_controller" filename="libgazebo_ros_gpu_laser.so">
         <topicName>/${robot_name}/scan</topicName>
-        <frameName>hokuyo_link</frameName>
+        <frameName>${prefix}_gpu_laser_link</frameName>
       </plugin>
     </sensor>

Commit message: refactor diffbot_description
- move stl files
- use separate robot.gazebo.xacro
- add addon xacro macro for addon components
- simplify wheel and motor macros: remove top level name from yaml files
- move caster macro to its own xacro file
- add camera sensor macro
- add imu sensor macro
- refactor gpu laser macro
- update license to BSDv3

File: diffbot_description/urdf/diffbot.urdf.xacro (robot description, xacro)
@@ -4,6 +4,7 @@
   <xacro:property name="robot_name" value="diffbot"/>
   <xacro:include filename="$(find ${package_name})/urdf/include/common_macros.urdf.xacro" />
+  <xacro:include filename="$(find ${package_name})/urdf/include/diffbot_caster_macro.urdf.xacro" />
   <xacro:include filename="$(find ${package_name})/urdf/include/common_sensors.xacro" />
-  <xacro:include filename="$(find ${package_name})/urdf/diffbot.gazebo.xacro" />
+  <xacro:include filename="$(find ${package_name})/urdf/include/robot.gazebo.xacro" />
   <xacro:property name="caster_wheel_yaml" value="$(find ${package_name})/config/${robot_name}/caster_wheel.yaml" />
   <xacro:property name="caster_wheel_props" value="${load_yaml(caster_wheel_yaml)}"/>
@@ -29,22 +30,18 @@
   <xacro:wheel prefix="front_right" reflect="-1"
                       wheel_props="${front_wheel_props}"
-                      base_props="${base_props}"
-                      mesh="${front_wheel_props['wheel']['mesh']}">
+                      base_props="${base_props}" >
   </xacro:wheel>
   <xacro:wheel prefix="front_left" reflect="1"
                       wheel_props="${front_wheel_props}"
-                      base_props="${base_props}"
-                      mesh="${front_wheel_props['wheel']['mesh']}">
+                      base_props="${base_props}" >
   </xacro:wheel>
   <!-- Motors -->
   <xacro:motor prefix="right" reflect="-1"
                       motor_props="${motor_props}"
-                      base_props="${base_props}"
-                      mesh="${motor_props['mesh']}">
+                      base_props="${base_props}" >
   </xacro:motor>
   <xacro:motor prefix="left" reflect="1"
                       motor_props="${motor_props}"
-                      base_props="${base_props}"
-                      mesh="${motor_props['mesh']}">
+                      base_props="${base_props}" >
   </xacro:motor>
   <!-- Sensors -->
@@ -52,3 +49,6 @@
                    sensor_prop="${sensor_prop}">
   </xacro:gpu_laser>
+  <!-- Gazebo -->
+  <xacro:gazebo_ros_control robotNamespace="/diffbot">
+  </xacro:gazebo_ros_control>
 </robot>

File: diffbot_description/urdf/include/common_macros.urdf.xacro (robot description, xacro)
@@ -16,25 +16,30 @@
 -->
   <xacro:macro name="wheel"
-               params="prefix reflect wheel_props base_props mesh:='' ">
+               params="prefix reflect wheel_props base_props ">
   <xacro:property name="pos_x_joint"
-     value="${(base_props['base']['x_size']/2) - wheel_props['wheel']['x_offset']}"/>
+     value="${(base_props['base']['x_size']/2) - wheel_props['x_offset']}"/>
   <xacro:property name="pos_y_joint"
-    value="${(base_props['base']['y_size']/2) + wheel_props['wheel']['y_offset'] + (wheel_props['wheel']['length']/2)}"/>
-  <xacro:property name="pos_z_joint" value="${wheel_props['wheel']['z_offset']}"/>
+    value="${(base_props['base']['y_size']/2) + wheel_props['y_offset'] + (wheel_props['length']/2)}"/>
+  <xacro:property name="pos_z_joint" value="${wheel_props['z_offset']}"/>
     <link name="${prefix}_wheel">
-    <xacro:if value="${mesh != '' }" >
+    <xacro:if value="${wheel_props['mesh'] != '' }" >
       <visual>
         <origin xyz="0.0 0 0" rpy="${pi/2} 0 ${pi/2.0*(reflect - 1)}"/>
         <geometry>
-          <mesh filename="package://${package_name}/meshes/${robot_name}/${mesh}" />
+          <xacro:if value="${wheel_props['scale'] == '' }" >
+            <mesh filename="package://${package_name}/meshes/${robot_name}/${wheel_props['mesh']}" />
+          </xacro:if>
+          <xacro:if value="${wheel_props['scale'] == '' }" >
+            <mesh filename="package://${package_name}/meshes/${robot_name}/${wheel_props['mesh']}" scale="${wheel_props['scale']}" />
+          </xacro:if>
         </geometry>
         <material name="dark_grey"/>
       </visual>
     </xacro:if>
-    <xacro:if value="${mesh == '' }" >
+    <xacro:if value="${wheel_props['mesh'] == '' }" >
       <visual>
         <origin xyz="0.0 0 0" rpy="${pi/2} 0 0"/>
          <geometry>
-         <cylinder radius="${wheel_props['wheel']['radius']}" length="${wheel_props['wheel']['length']}"/>
+         <cylinder radius="${wheel_props['radius']}" length="${wheel_props['length']}"/>
         </geometry>
         <material name="red"/>
@@ -44,10 +49,10 @@
         <origin xyz="0 0 0" rpy="${pi/2} 0 0"/>
         <geometry>
-          <cylinder radius="${wheel_props['wheel']['radius']}" length="${wheel_props['wheel']['length']}"/>
+          <cylinder radius="${wheel_props['radius']}" length="${wheel_props['length']}"/>
         </geometry>
       </collision>
-      <xacro:cylinder_inertia m="${wheel_props['wheel']['mass']}"
-                              r="${wheel_props['wheel']['radius']}"
-                              l="${wheel_props['wheel']['length']}"
+      <xacro:cylinder_inertia m="${wheel_props['mass']}"
+                              r="${wheel_props['radius']}"
+                              l="${wheel_props['length']}"
                               o_xyz="0.0 0.0 0.0"
                               o_rpy="${pi/2.0} 0.0 0.0" >
@@ -74,143 +79,4 @@
     </transmission>
   </xacro:macro>
-<!-- ======================================================================= -->
-<!-- Caster wheel link & joint macro -->
-  <!-- locationprefix locationright wheel_base_dx TODO remove -->
-  <xacro:macro name="caster_wheel"
-                params="prefix reflect wheel_props locationright:=${0} ">
-    <!-- caster base (fixed) -->
-    <link name="${prefix}_caster_base_link">
-      <xacro:box_inertia  m="${wheel_props['base']['mass']}"
-                          x="${wheel_props['base']['size']['x']}"
-                          y="${wheel_props['base']['size']['y']}"
-                          z="${wheel_props['base']['size']['z']}"
-                          o_xyz="0.0 0.0 ${-wheel_props['base']['size']['z']/2.0}"
-                          o_rpy="0.0 0.0 0.0" />
-      <xacro:if value="${wheel_props['base']['mass'] != '' }" >
-        <visual>
-            <origin xyz="0 0 ${-wheel_props['base']['size']['z']/2.0}" rpy="0 0 0" />
-            <geometry>
-                <mesh filename="package://${package_name}/meshes/${robot_name}/${wheel_props['base']['mesh']}" />
-            </geometry>
-            <!-- xacro:insert_block name="material_silver" / TODO use this block? -->
-            <material name="silver"/>
-        </visual>
-      </xacro:if>
-      <xacro:if value="${wheel_props['base']['mass'] == '' }" >
-        <visual>
-          <origin xyz="0 0 ${-wheel_props['base']['size']['z']/2.0}" rpy="0 0 0" />
-          <geometry>
-            <box size="${wheel_props['base']['size']['x']} ${wheel_props['base']['size']['y']} ${wheel_props['base']['size']['z']}" />
-          </geometry>
-          <material name="red"/>
-        </visual>
-      </xacro:if>
-      <collision>
-        <origin xyz="0 0 ${-wheel_props['base']['size']['z']/2.0}" rpy="0 0 0" />
-        <geometry>
-          <box size="${wheel_props['base']['size']['x']} ${wheel_props['base']['size']['y']} ${wheel_props['base']['size']['z']}" />
-        </geometry>
-      </collision>
-    </link>
-    <joint name="${prefix}_caster_base_joint" type="fixed">
-      <origin xyz="${wheel_props['base']['dx']} ${-wheel_props['base']['dy'] * locationright} ${wheel_props['base']['dz']}"
-              rpy="0 0 0" />
-      <parent link="base_link" />
-      <child link="${prefix}_caster_base_link" />
-      <axis xyz="0 0 1" />
-      <dynamics damping="0.01" friction="0.0"/>
-    </joint>
-    <gazebo reference="${prefix}_caster_base_link">
-      <material>Gazebo/Grey</material>
-    </gazebo>
-    <!-- caster hub -->
-    <link name="${prefix}_caster_rotation_link">
-      <xacro:box_inertia  m="${wheel_props['hub']['mass']}"
-                          x="${wheel_props['hub']['size']['x']}"
-                          y="${wheel_props['hub']['size']['y']}"
-                          z="${wheel_props['hub']['size']['z']}"
-                          o_xyz="0.0 0.0 ${-wheel_props['hub']['size']['z']/2.0}"
-                          o_rpy="0.0 0.0 0.0" />
-      <xacro:if value="${wheel_props['hub']['mesh'] != '' }" >
-        <visual>
-          <origin xyz="0 0 ${-wheel_props['hub']['size']['z']/2.0}" rpy="0 0 0" />
-          <geometry>
-            <mesh filename="package://${package_name}/meshes/${robot_name}/${wheel_props['hub']['mesh']}" />
-          </geometry>
-          <!-- xacro:insert_block name="material_silver" / TODO use this block? -->
-          <material name="silver"/>
-        </visual>
-      </xacro:if>
-      <xacro:if value="${wheel_props['hub']['mesh'] == '' }" >
-        <visual>
-          <origin xyz="0 0 ${-wheel_props['hub']['size']['z']/2.0}" rpy="0 0 0" />
-          <geometry>
-            <box size="${wheel_props['hub']['size']['x']} ${wheel_props['hub']['size']['y']} ${wheel_props['hub']['size']['z']}" />
-          </geometry>
-          <material name="red"/>
-        </visual>
-      </xacro:if>
-      <collision>
-        <origin xyz="0 0 ${-wheel_props['hub']['size']['z']/2.0}" rpy="0 0 0" />
-        <geometry>
-          <box size="${wheel_props['hub']['size']['x']} ${wheel_props['hub']['size']['y']} ${wheel_props['hub']['size']['z']}" />
-        </geometry>
-      </collision>
-    </link>
-    <joint name="${prefix}_caster_rotation_joint" type="continuous">
-      <origin xyz="${wheel_props['hub']['dx']} ${-wheel_props['hub']['dy'] * locationright} ${wheel_props['hub']['dz']}"
-              rpy="0 0 0" />
-      <parent link="base_link" />
-      <child link="${prefix}_caster_rotation_link" />
-      <axis xyz="0 0 1" />
-      <dynamics damping="0.01" friction="0.0"/>
-    </joint>
-    <gazebo reference="${prefix}_caster_rotation_link">
-      <material>Gazebo/Grey</material>
-    </gazebo>
-    <!-- caster wheel -->
-    <link name="${prefix}_caster_wheel_link">
-      <xacro:cylinder_inertia m="${wheel_props['wheel']['mass']}"
-                              r="${wheel_props['wheel']['radius']}"
-                              l="${wheel_props['wheel']['length']}">
-        <!-- TODO unused block error?: origin xyz="0 0 0" rpy="${pi/2} 0 0" /-->
-      </xacro:cylinder_inertia>
-      <xacro:if value="${wheel_props['wheel']['mesh'] != '' }" >
-        <visual>
-          <origin xyz="0 0 0" rpy="0 0 0" />
-          <geometry>
-            <mesh filename="package://${package_name}/meshes/${robot_name}/${wheel_props['wheel']['mesh']}" />
-          </geometry>
-          <!-- TODO use this?: xacro:insert_block name="material_dark_grey" /-->
-          <material name="dark_grey"/>
-        </visual>
-      </xacro:if>
-      <xacro:if value="${wheel_props['wheel']['mesh'] == '' }" >
-        <visual>
-          <origin xyz="0 0 0" rpy="${pi/2} 0 0" />
-          <geometry>
-            <cylinder length="${wheel_props['wheel']['length']}" radius="${wheel_props['wheel']['radius']}" />
-          </geometry>
-          <material name="red"/>
-        </visual>
-      </xacro:if>
-      <collision>
-        <origin xyz="0 0 0" rpy="${pi/2} 0 0" />
-        <geometry>
-          <cylinder length="${wheel_props['wheel']['length']}" radius="${wheel_props['wheel']['radius']}" />
-        </geometry>
-      </collision>
-    </link>
-    <joint name="${prefix}_caster_wheel_joint" type="continuous">
-      <origin xyz="${wheel_props['wheel']['dx']} ${-wheel_props['wheel']['dy'] * locationright} ${wheel_props['wheel']['dz']}"
-              rpy="0 0 0" />
-      <parent link="${prefix}_caster_rotation_link" />
-      <child link="${prefix}_caster_wheel_link" />
-      <axis xyz="0 1 0" />
-    </joint>
-    <gazebo reference="${prefix}_caster_wheel_link">
-      <material>Gazebo/DarkGrey</material>
-    </gazebo>
-  </xacro:macro>
 <!-- ===================== Motor xacro =========================================
   Xacro to create a motor link and the respective joint. For more detail information and usage, see:
@@ -225,5 +91,5 @@
 -->
   <xacro:macro name="motor"
-               params="prefix reflect motor_props base_props mesh:='' ">
+               params="prefix reflect motor_props base_props ">
   <xacro:property name="pos_x_joint"
      value="${(base_props['base']['x_size']/2) - motor_props['x_offset']}"/>
@@ -232,14 +98,19 @@
   <xacro:property name="pos_z_joint" value="${motor_props['z_offset']}"/>
     <link name="${prefix}_motor">
-    <xacro:if value="${mesh != '' }" >
+    <xacro:if value="${motor_props['mesh'] != '' }" >
       <visual>
         <origin xyz="0.0 0.0 0.0" rpy="0.0 0 ${pi/2.0*(reflect - 1)}"/>
         <geometry>
-          <mesh filename="package://${package_name}/meshes/${robot_name}/${mesh}" />
+          <xacro:if value="${motor_props['scale'] == '' }" >
+            <mesh filename="package://${package_name}/meshes/${robot_name}/${motor_props['mesh']}" />
+          </xacro:if>
+          <xacro:if value="${motor_props['scale'] == '' }" >
+            <mesh filename="package://${package_name}/meshes/${robot_name}/${motor_props['mesh']}" scale="${motor_props['scale']}"/>
+          </xacro:if>
         </geometry>
         <material name="blue"/>
       </visual>
     </xacro:if>
-    <xacro:if value="${mesh == '' }" >
+    <xacro:if value="${motor_props['mesh'] == '' }" >
       <visual>
         <origin xyz="0.0 0 0" rpy="${pi/2} 0 0"/>
@@ -285,5 +156,5 @@
 -->
   <xacro:macro name="base"
-               params="base_prop mesh:='' *origin ">
+               params="base_prop mesh:='' scale:='' *origin ">
     <link name="base_link">
     <xacro:box_inertia m="${base_prop['base']['mass']}"
@@ -297,5 +168,10 @@
         <geometry>
           <!-- The folder path get a folder_name global parameter -->
-          <mesh filename="package://${package_name}/meshes/${robot_name}/${mesh}" />
+          <xacro:if value="${scale != '' }" >
+            <mesh filename="package://${package_name}/meshes/${robot_name}/${mesh}" scale="${scale}"/>
+          </xacro:if>
+          <xacro:if value="${scale == '' }" >
+            <mesh filename="package://${package_name}/meshes/${robot_name}/${mesh}" />
+          </xacro:if>
         </geometry>
         <material name="white" />
@@ -338,6 +214,6 @@
       <child link="base_link" />
       <!-- origin xyz="0 0 ${wheel_radius - base_z_origin_to_wheel_origin}" rpy="0 0 0" /-->
-      <!-- origin xyz="0 0 ${wheel_props['wheel']['radius'] - wheel_props['wheel']['z_offset'] + 0.1}" rpy="0 0 0" /-->
-      <origin xyz="0 0 ${wheel_props['wheel']['radius'] - wheel_props['wheel']['z_offset']}" rpy="0 0 0" />
+      <!-- origin xyz="0 0 ${wheel_props['radius'] - wheel_props['z_offset'] + 0.1}" rpy="0 0 0" /-->
+      <origin xyz="0 0 ${wheel_props['radius'] - wheel_props['z_offset']}" rpy="0 0 0" />
     </joint>
   </xacro:macro>
