Commit message: refactor diffbot_description
- move stl files
- use separate robot.gazebo.xacro
- add addon xacro macro for addon components
- simplify wheel and motor macros: remove top level name from yaml files
- move caster macro to its own xacro file
- add camera sensor macro
- add imu sensor macro
- refactor gpu laser macro
- update license to BSDv3

File: diffbot_description/urdf/include/common_sensors.xacro (robot description, xacro)
@@ -5,34 +5,33 @@
      value="${sensor_prop['gpu_laser']['mesh']}"/>
   <link name="${prefix}_gpu_laser_link">
-      <xacro:if value="${mesh != '' }" >
-      <visual>
-        <origin xyz="0 0 0" rpy="0 0 0"/>
-        <geometry>
-          <mesh filename="package://${package_name}/meshes/sensors/${mesh}" />
-        </geometry>
-        <material name="dark_grey"/>
-      </visual>
-    </xacro:if>
-    <xacro:if value="${mesh == '' }" >
-      <visual>
-        <origin xyz="0 0 0" rpy="0 0 0"/>
-         <geometry>
-         <cylinder radius="${sensor_prop['gpu_laser']['radius']}" length="${sensor_prop['gpu_laser']['length']}"/>
-        </geometry>
-        <material name="red"/>
-      </visual>
-    </xacro:if>
-      <collision>
-        <origin xyz="0 0 0" rpy="0 0 0"/>
-        <geometry>
-          <cylinder radius="${sensor_prop['gpu_laser']['radius']}" length="${sensor_prop['gpu_laser']['length']}"/>
-        </geometry>
-      </collision>
-      <xacro:cylinder_inertia m="${sensor_prop['gpu_laser']['mass']}"
-                              r="${sensor_prop['gpu_laser']['radius']}"
-                              l="${sensor_prop['gpu_laser']['length']}"
-                              o_xyz="0 0 0"
-                              o_rpy="0 0 0" >
-      </xacro:cylinder_inertia>
+    <xacro:if value="${mesh != '' }" >
+    <visual>
+      <origin xyz="0 0 0" rpy="0 0 0"/>
+      <geometry>
+        <mesh filename="package://${package_name}/meshes/sensors/${mesh}" />
+      </geometry>
+      <material name="dark_grey"/>
+    </visual>
+  </xacro:if>
+  <xacro:if value="${mesh == '' }" >
+    <visual>
+      <origin xyz="0 0 0" rpy="0 0 0"/>
+        <geometry>
+        <cylinder radius="${sensor_prop['gpu_laser']['radius']}" length="${sensor_prop['gpu_laser']['length']}"/>
+      </geometry>
+      <material name="red"/>
+    </visual>
+  </xacro:if>
+    <collision>
+      <origin xyz="0 0 0" rpy="0 0 0"/>
+      <geometry>
+        <cylinder radius="${sensor_prop['gpu_laser']['radius']}" length="${sensor_prop['gpu_laser']['length']}"/>
+      </geometry>
+    </collision>
+    <xacro:cylinder_inertia m="${sensor_prop['gpu_laser']['mass']}"
+                            r="${sensor_prop['gpu_laser']['radius']}"
+                            l="${sensor_prop['gpu_laser']['length']}"
+                            o_xyz="0 0 0"
+                            o_rpy="0 0 0" />
   </link>
   <gazebo reference="${prefix}_gpu_laser_link">
@@ -82,3 +81,152 @@
   </gazebo>
 </xacro:macro>
+<xacro:macro name="camera_sensor" params=" *joint_origin parent_link sensor_prop visualize mesh:='' ">
+  <link name="camera_link">
+    <xacro:if value="${mesh != '' }" >
+      <visual>
+        <origin xyz="0 0 0" rpy="0 0 0"/>
+        <geometry>
+          <mesh filename="package://${package_name}/meshes/sensors/${mesh}" scale="${sensor_prop['camera']['meshes']['scale']}" />
+        </geometry>
+        <material name="dark_grey"/>
+      </visual>
+    </xacro:if>
+    <xacro:if value="${mesh == '' }" >
+      <visual>
+        <origin xyz="0 0 0" rpy="0 0 0"/>
+        <geometry>
+          <cylinder radius="${sensor_prop['camera']['radius']}" length="${sensor_prop['camera']['length']}"/>
+        </geometry>
+        <material name="red"/>
+      </visual>
+    </xacro:if>
+    <collision>
+      <origin xyz="0 0 0" rpy="0 0 0"/>
+      <geometry>
+        <cylinder radius="0.03" length="0.03"/>
+      </geometry>
+    </collision>
+    <xacro:cylinder_inertia m="${sensor_prop['camera']['mass']}"
+                            r="${sensor_prop['camera']['radius']}"
+                            l="${sensor_prop['camera']['length']}"
+                            o_xyz="0 0 0"
+                            o_rpy="0 0 0" />
+  </link>
+  <gazebo reference="camera_link">
+    <material>Gazebo/Red</material>
+  </gazebo>
+  <joint name="camera_joint" type="fixed">
+    <axis xyz="0 1 0" />
+    <xacro:insert_block name="joint_origin" />
+    <parent link="${parent_link}"/>
+    <child link="camera_link"/>
+  </joint>
+  <gazebo reference="camera_link">
+    <sensor type="camera" name="camera1">
+      <update_rate>60</update_rate>
+      <visualize>${visualize}</visualize>
+      <camera>
+        <horizontal_fov>1.92</horizontal_fov>
+        <image>
+          <width>640</width>
+          <height>480</height>
+          <format>B8G8R8</format>
+        </image>
+        <depth_camera>
+        </depth_camera>
+        <clip>
+          <near>0.02</near>
+          <far>300</far>
+        </clip>
+        <noise>
+          <type>gaussian</type>
+          <!-- Noise is sampled independently per pixel on each frame.
+                That pixel's noise value is added to each of its color
+                channels, which at that point lie in the range [0,1]. -->
+          <mean>0.0</mean>
+          <stddev>0.007</stddev>
+        </noise>
+      </camera>
+      <plugin name="camera_controller" filename="libgazebo_ros_camera.so">
+        <ros>
+          <!-- <namespace>/</namespace> -->
+          <!-- topics need to be prefixed with camera_name for remapping -->
+          <!-- <remapping>image_raw:=image_demo</remapping> -->
+        </ros>
+        <!-- omit camera_name to default to sensor name -->
+        <!-- <camera_name>mycamera</camera_name> -->
+        <!-- frame_name>omit so it defaults to link name</frame_name-->
+      </plugin>
+    </sensor>
+  </gazebo>
+</xacro:macro>
+<xacro:macro name="imu_sensor" params=" *joint_origin parent_link sensor_prop">
+  <xacro:property name="mesh"
+     value="${sensor_prop['imu']['mesh']}"/>
+  <link name="imu_link">
+    <xacro:if value="${mesh != '' }" >
+      <visual>
+        <origin xyz="0 0 0" rpy="0 0 0"/>
+        <geometry>
+          <mesh filename="package://${package_name}/meshes/sensors/${mesh}" scale="${sensor_prop['imu']['scale']}" />
+        </geometry>
+        <material name="dark_grey"/>
+      </visual>
+    </xacro:if>
+    <xacro:if value="${mesh == '' }" >
+      <visual>
+        <origin xyz="0 0 0" rpy="0 0 0"/>
+        <geometry>
+          <cylinder radius="${sensor_prop['imu']['radius']}" length="${sensor_prop['imu']['length']}"/>
+        </geometry>
+        <material name="red"/>
+      </visual>
+    </xacro:if>
+    <collision>
+      <origin xyz="0 0 0" rpy="0 0 0"/>
+      <geometry>
+        <box size="0.01 0.01 0.01"/>
+      </geometry>
+    </collision>
+    <xacro:box_inertia m="${sensor_prop['imu']['mass']}"
+                       x="${sensor_prop['imu']['size']['x']}"
+                       y="${sensor_prop['imu']['size']['y']}"
+                       z="${sensor_prop['imu']['size']['y']}" />
+    <!-- Todo delete visual>
+      <origin xyz="0 0 0" rpy="0 0 0"/>
+      <geometry>
+        <box size="0.01 0.01 0.01"/>
+      </geometry>
+    </visual>
+    <inertial>
+      <mass value="1e-5" />
+      <origin xyz="0 0 0" rpy="0 0 0"/>
+      <inertia ixx="1e-6" ixy="0" ixz="0" iyy="1e-6" iyz="0" izz="1e-6" />
+    </inertial-->
+  </link>
+  <gazebo reference="imu_link">
+    <material>Gazebo/Yellow</material>
+  </gazebo>
+  <joint name="imu_joint" type="fixed">
+    <axis xyz="0 1 0" />
+    <xacro:insert_block name="joint_origin" />
+    <parent link="${parent_link}"/>
+    <child link="imu_link"/>
+  </joint>
+  <gazebo reference="imu_link">
+    <sensor type="imu" name="my_imu">
+    <always_on>true</always_on>
+    <!-- Publish at 30 hz -->
+    <update_rate>30</update_rate>
+    <plugin name="my_imu_plugin" filename="libgazebo_ros_imu_sensor.so">
+      <ros>
+        <!-- Will publish to /imu/data -->
+        <namespace>/imu</namespace>
+        <argument>~/out:=data</argument>
+      </ros>
+      <!-- frame_name ommited, will be "my_link" -->
+    </plugin>
+    </sensor>
+  </gazebo>
+</xacro:macro>
 </robot>

File: diffbot_description/urdf/include/robot.gazebo.xacro (robot description, xacro)
@@ -2,11 +2,13 @@
 <robot xmlns:xacro="http://ros.org/wiki/xacro">
   <!-- ros_control plugin -->
-  <gazebo>
-    <plugin name="gazebo_ros_control" filename="libgazebo_ros_control.so">
-      <robotNamespace>/diffbot</robotNamespace>
-      <!--robotParam>/robot_description</robotParam-->
-      <robotSimType>gazebo_ros_control/DefaultRobotHWSim</robotSimType>
-    </plugin>
-  </gazebo>
+  <xacro:macro name="gazebo_ros_control" params="robotNamespace robotSimType:=gazebo_ros_control/DefaultRobotHWSim">
+    <gazebo>
+      <plugin name="gazebo_ros_control" filename="libgazebo_ros_control.so">
+        <robotNamespace>${robotNamespace}</robotNamespace>
+        <!--robotParam>/robot_description</robotParam-->
+        <robotSimType>${robotSimType}</robotSimType>
+      </plugin>
+    </gazebo>
+  </xacro:macro>
   <!-- xacro to set the friction for the wheel. This patch was taken from the MIR
   repository.

Commit message: update diffbot_description: add gpu arg for laser xacro macro (#27)

File: diffbot_description/urdf/diffbot.urdf.xacro (robot description, xacro)
@@ -46,7 +46,7 @@
   </xacro:motor>
   <!-- Sensors -->
-  <xacro:gpu_laser prefix="rplidar" parent_link="base_link"
+  <xacro:laser prefix="rplidar" parent_link="base_link"
                    sensor_prop="${sensor_prop}">
-  </xacro:gpu_laser>
+  </xacro:laser>
   <!-- Gazebo -->
   <xacro:gazebo_ros_control robotNamespace="/diffbot">

File: diffbot_description/urdf/include/common_sensors.xacro (robot description, xacro)
@@ -1,11 +1,19 @@
 <?xml version="1.0"?>
 <robot xmlns:xacro="http://www.ros.org/wiki/xacro">
-<xacro:macro name="gpu_laser" params="prefix parent_link sensor_prop ">
+<xacro:macro name="laser" params="prefix parent_link sensor_prop enable_gpu:=true">
   <xacro:property name="mesh"
-     value="${sensor_prop['gpu_laser']['mesh']}"/>
-  <link name="${prefix}_gpu_laser_link">
+     value="${sensor_prop['laser']['mesh']}"/>
+  <xacro:if value="${enable_gpu}">
+    <xacro:property name="plugin_name" value="libgazebo_ros_gpu_laser.so"/>
+    <xacro:property name="laser_type" value="gpu_ray"/>
+  </xacro:if>
+  <xacro:if value="${not enable_gpu}">
+    <xacro:property name="plugin_name" value="libgazebo_ros_laser.so"/>
+    <xacro:property name="laser_type" value="ray"/>
+  </xacro:if>
+  <link name="${prefix}_laser_link">
     <xacro:if value="${mesh != '' }" >
     <visual>
-      <origin xyz="0 0 0" rpy="0 0 0"/>
+      <origin xyz="0 0 0" rpy="0 0 ${pi}"/>
       <geometry>
         <mesh filename="package://${package_name}/meshes/sensors/${mesh}" />
@@ -18,5 +26,5 @@
       <origin xyz="0 0 0" rpy="0 0 0"/>
         <geometry>
-        <cylinder radius="${sensor_prop['gpu_laser']['radius']}" length="${sensor_prop['gpu_laser']['length']}"/>
+        <cylinder radius="${sensor_prop['laser']['radius']}" length="${sensor_prop['laser']['length']}"/>
       </geometry>
       <material name="red"/>
@@ -26,35 +34,36 @@
       <origin xyz="0 0 0" rpy="0 0 0"/>
       <geometry>
-        <cylinder radius="${sensor_prop['gpu_laser']['radius']}" length="${sensor_prop['gpu_laser']['length']}"/>
+        <cylinder radius="${sensor_prop['laser']['radius']}" length="${sensor_prop['laser']['length']}"/>
       </geometry>
     </collision>
-    <xacro:cylinder_inertia m="${sensor_prop['gpu_laser']['mass']}"
-                            r="${sensor_prop['gpu_laser']['radius']}"
-                            l="${sensor_prop['gpu_laser']['length']}"
+    <xacro:cylinder_inertia m="${sensor_prop['laser']['mass']}"
+                            r="${sensor_prop['laser']['radius']}"
+                            l="${sensor_prop['laser']['length']}"
                             o_xyz="0 0 0"
                             o_rpy="0 0 0" />
   </link>
   <gazebo reference="${prefix}_laser_link">
-    <material>Gazebo/Grey</material>
-  </gazebo>
-  <joint name="${prefix}_gpu_laser_joint" type="fixed">
+    <material>${sensor_prop['laser']['color']}</material>
+  </gazebo>
+  <joint name="${prefix}_laser_joint" type="fixed">
     <parent link="${parent_link}"/>
-    <child link="${prefix}_gpu_laser_link"/>
-    <origin xyz="${sensor_prop['gpu_laser']['dx']} ${sensor_prop['gpu_laser']['dy']} ${sensor_prop['gpu_laser']['dz']}" rpy="0 0 0"/>
+    <child link="${prefix}_laser_link"/>
+    <origin xyz="${sensor_prop['laser']['dx']} ${sensor_prop['laser']['dy']} ${sensor_prop['laser']['dz']}" rpy="0 0 ${pi}"/>
     <axis xyz="0 1 0" />
   </joint>
   <!-- hokuyo gazebo references -->
-  <gazebo reference="${prefix}_gpu_laser_link">
-    <sensor type="gpu_ray" name="head_hokuyo_sensor">
+  <gazebo reference="${prefix}_laser_link">
+    <!-- type is either gpu_laser or laser -->
+    <sensor type="${laser_type}" name="head_hokuyo_sensor">
       <pose>0 0 0 0 0 0</pose>
       <visualize>true</visualize>
-      <update_rate>40</update_rate>
+      <update_rate>12</update_rate>
       <ray>
         <scan>
           <horizontal>
-            <samples>720</samples>
+            <samples>360</samples>
             <resolution>1</resolution>
-            <min_angle>${sensor_prop['gpu_laser']['angular_range']['min']}</min_angle>
-            <max_angle>${sensor_prop['gpu_laser']['angular_range']['max']}</max_angle>
+            <min_angle>${sensor_prop['laser']['angular_range']['min']}</min_angle>
+            <max_angle>${sensor_prop['laser']['angular_range']['max']}</max_angle>
           </horizontal>
         </scan>
@@ -74,7 +83,8 @@
         </noise>
       </ray>
-      <plugin name="gazebo_ros_head_hokuyo_controller" filename="libgazebo_ros_gpu_laser.so">
-        <topicName>/${robot_name}/scan</topicName>
-        <frameName>${prefix}_gpu_laser_link</frameName>
+      <!-- plugin_name is either libgazebo_ros_laser.so or libgazebo_ros_gpu_laser.so-->
+      <plugin name="gazebo_ros_head_hokuyo_controller" filename="${plugin_name}">
+        <topicName>/diffbot/scan</topicName>
+        <frameName>${prefix}_laser_link</frameName>
       </plugin>
     </sensor>

Commit message: fix deprecated warning using load_yaml (#53)
Using xacro.load_yaml instead of just load_yaml

File: diffbot_description/urdf/diffbot.urdf.xacro (robot description, xacro)
@@ -8,13 +8,13 @@
   <xacro:include filename="$(find ${package_name})/urdf/include/robot.gazebo.xacro" />
   <xacro:property name="caster_wheel_yaml" value="$(find ${package_name})/config/${robot_name}/caster_wheel.yaml" />
-  <xacro:property name="caster_wheel_props" value="${load_yaml(caster_wheel_yaml)}"/>
+  <xacro:property name="caster_wheel_props" value="${xacro.load_yaml(caster_wheel_yaml)}"/>
   <xacro:property name="front_wheel_yaml" value="$(find ${package_name})/config/${robot_name}/front_wheel.yaml" />
-  <xacro:property name="front_wheel_props" value="${load_yaml(front_wheel_yaml)}"/>
+  <xacro:property name="front_wheel_props" value="${xacro.load_yaml(front_wheel_yaml)}"/>
   <xacro:property name="motor_yaml" value="$(find ${package_name})/config/${robot_name}/motor.yaml" />
-  <xacro:property name="motor_props" value="${load_yaml(motor_yaml)}"/>
+  <xacro:property name="motor_props" value="${xacro.load_yaml(motor_yaml)}"/>
   <xacro:property name="base_yaml" value="$(find ${package_name})/config/${robot_name}/base.yaml" />
-  <xacro:property name="base_props" value="${load_yaml(base_yaml)}"/>
+  <xacro:property name="base_props" value="${xacro.load_yaml(base_yaml)}"/>
   <xacro:property name="sensor_yaml" value="$(find ${package_name})/config/${robot_name}/sensors.yaml" />
-  <xacro:property name="sensor_prop" value="${load_yaml(sensor_yaml)}"/>
+  <xacro:property name="sensor_prop" value="${xacro.load_yaml(sensor_yaml)}"/>
   <!-- Footprint link -->
   <xacro:footprint wheel_props="${front_wheel_props}" />

Commit message: Changes related to sbc BNO055 IMU

File: diffbot_description/urdf/diffbot.urdf.xacro (robot description, xacro)
@@ -8,13 +8,13 @@
   <xacro:include filename="$(find ${package_name})/urdf/include/robot.gazebo.xacro" />
   <xacro:property name="caster_wheel_yaml" value="$(find ${package_name})/config/${robot_name}/caster_wheel.yaml" />
-  <xacro:property name="caster_wheel_props" value="${xacro.load_yaml(caster_wheel_yaml)}"/>
+  <xacro:property name="caster_wheel_props" value="${load_yaml(caster_wheel_yaml)}"/>
   <xacro:property name="front_wheel_yaml" value="$(find ${package_name})/config/${robot_name}/front_wheel.yaml" />
-  <xacro:property name="front_wheel_props" value="${xacro.load_yaml(front_wheel_yaml)}"/>
+  <xacro:property name="front_wheel_props" value="${load_yaml(front_wheel_yaml)}"/>
   <xacro:property name="motor_yaml" value="$(find ${package_name})/config/${robot_name}/motor.yaml" />
-  <xacro:property name="motor_props" value="${xacro.load_yaml(motor_yaml)}"/>
+  <xacro:property name="motor_props" value="${load_yaml(motor_yaml)}"/>
   <xacro:property name="base_yaml" value="$(find ${package_name})/config/${robot_name}/base.yaml" />
-  <xacro:property name="base_props" value="${xacro.load_yaml(base_yaml)}"/>
+  <xacro:property name="base_props" value="${load_yaml(base_yaml)}"/>
   <xacro:property name="sensor_yaml" value="$(find ${package_name})/config/${robot_name}/sensors.yaml" />
-  <xacro:property name="sensor_prop" value="${xacro.load_yaml(sensor_yaml)}"/>
+  <xacro:property name="sensor_prop" value="${load_yaml(sensor_yaml)}"/>
   <!-- Footprint link -->
   <xacro:footprint wheel_props="${front_wheel_props}" />
@@ -53,3 +53,11 @@
   <xacro:gazebo_ros_control robotNamespace="/diffbot">
   </xacro:gazebo_ros_control>
+  <joint name="imu_sensor_joint" type="fixed">
+    <parent link="base_link"/>
+    <child link="imu_sensor_link"/>
+    <origin xyz="0.0 -0.01 0.00"/>
+    <axis xyz="0 0 0"/>
+  </joint>
+  <link name="imu_sensor_link">
+  </link>
 </robot>
