Commit message: Frames: base_link and base_footprint at the axle's midpoint
diff_drive_controller computes the odometry for the midpoint between the drive
wheels and publishes it as base_footprint. That frame was below the center of
DiffBot's base plate, 18.5 mm behind the axle (Remo's was 36 mm), so during a
turn on the spot TF put the robot and its sensors on a small arc that the real
robot doesn't drive.

- DiffBot's URDF: base_link is the axle's midpoint, with base_footprint on the
  ground below it, as before. The base plate and every part attached to it are
  defined around a new chassis_link, 18.5 mm behind base_link, so no part moves
  relative to the others.
- remo_description is pinned to its matching change.
- Navigation: each robot has its own costmap footprint in
  diffbot_navigation/config/<model>/, around the new origin and covering the
  whole model, which the shared rectangle didn't (DiffBot's rear and wheels
  were outside it). move_base and Move Base Flex load it with the model argument.
- The simulation test: base_footprint now moves less than 1 mm during the turn,
  so the check tightens from 0.15 m to 0.02 m.

File: diffbot_description/urdf/diffbot.urdf.xacro (robot description, xacro)
@@ -19,6 +19,8 @@
   <!-- Footprint link -->
   <xacro:footprint wheel_props="${front_wheel_props}" />
-  <!-- Base link -->
-  <xacro:base base_prop="${base_props}" mesh="${base_props['base']['mesh']}" >
+  <!-- Base link at the drive axle's midpoint, and the chassis around it. The wheels sit
+       x_offset behind the base plate's front edge, the same position the wheel macro uses -->
+  <xacro:property name="axle_x" value="${base_props['base']['x_size']/2 - front_wheel_props['x_offset']}"/>
+  <xacro:base base_prop="${base_props}" axle_x="${axle_x}" mesh="${base_props['base']['mesh']}" >
     <origin xyz="0 0 0" rpy="0 0 0" />
   </xacro:base>
@@ -46,5 +48,5 @@
   </xacro:motor>
   <!-- Sensors -->
-  <xacro:laser prefix="rplidar" parent_link="base_link"
+  <xacro:laser prefix="rplidar" parent_link="chassis_link"
                    sensor_prop="${sensor_prop}"
                    enable_gpu="${sensor_prop['laser']['enable_gpu']}">

File: diffbot_description/urdf/include/common_macros.urdf.xacro (robot description, xacro)
@@ -68,5 +68,5 @@
     <joint name="${prefix}_wheel_joint" type="continuous">
       <axis xyz="0 1 0" rpy="0 0 0" />
-      <parent link="base_link"/>
+      <parent link="chassis_link"/>
       <child link="${prefix}_wheel"/>
       <origin xyz="${pos_x_joint} ${reflect* pos_y_joint} ${pos_z_joint}" rpy="0 0 0"/>
@@ -138,5 +138,5 @@
     </link>
     <joint name="${prefix}_motor_joint" type="fixed">
-      <parent link="base_link"/>
+      <parent link="chassis_link"/>
       <child link="${prefix}_motor"/>
       <origin xyz="${pos_x_joint} ${reflect* pos_y_joint} ${pos_z_joint}" rpy="0 ${-pi/2.0*(reflect - 1)} 0"/>
@@ -155,4 +155,6 @@
   params:
   - base_props [dictionary]: base link properties;
+  - axle_x [float]: how far the drive axle's midpoint (base_link) lies in front of the base
+    plate's center (chassis_link), in m;
   - mesh [string]: file name of the link mesh;
     - DEFAULT Value -> Empty string
@@ -160,6 +162,16 @@
 -->
   <xacro:macro name="base"
-               params="base_prop mesh:='' scale:='' *origin ">
-    <link name="base_link">
+               params="base_prop axle_x mesh:='' scale:='' *origin ">
+    <!-- base_link is the robot's reference frame: the midpoint between the drive wheels, where
+         diff_drive_controller's odometry puts the robot. The chassis' geometry, mass and all
+         attached parts are defined around chassis_link, the center of the base plate, which lies
+         axle_x behind it. -->
+    <link name="base_link" />
+    <joint name="chassis_joint" type="fixed">
+      <parent link="base_link"/>
+      <child link="chassis_link"/>
+      <origin xyz="${-axle_x} 0 0" rpy="0 0 0"/>
+    </joint>
+    <link name="chassis_link">
     <xacro:box_inertia m="${base_prop['base']['mass']}"
                        x="${base_prop['base']['x_size']}"

File: diffbot_description/urdf/include/diffbot_caster_macro.urdf.xacro (robot description, xacro)
@@ -58,5 +58,5 @@
       <origin xyz="${wheel_props['base']['dx']} ${-wheel_props['base']['dy'] * locationright} ${wheel_props['base']['dz']}"
               rpy="0 0 0" />
-      <parent link="base_link" />
+      <parent link="chassis_link" />
       <child link="${prefix}_caster_base_link" />
       <axis xyz="0 0 1" />
@@ -108,5 +108,5 @@
       <origin xyz="${wheel_props['hub']['dx']} ${-wheel_props['hub']['dy'] * locationright} ${wheel_props['hub']['dz']}"
               rpy="0 0 0" />
-      <parent link="base_link" />
+      <parent link="chassis_link" />
       <child link="${prefix}_caster_rotation_link" />
       <axis xyz="0 0 1" />

Commit message: Simulation: an IMU in Gazebo for DiffBot and Remo, as the robot publishes it
DiffBot's model gets the same IMU macro as Remo's in remo_description 2.1.0: imu_link on chassis_link with Gazebo's ROS 1 IMU plugin at 50 Hz (the old macro had ROS 2 plugin syntax, which Gazebo Classic ignores, and inconsistent sizes). DiffBot has no IMU on the robot, so its simulated one weighs 1 g and its position is a placeholder (xacro arguments imu_xyz and imu_rpy). An adapter node republishes the plugin's imu/gazebo as imu/data_raw without the orientation, as the firmware publishes it. A new test in both robots' simulation tests checks the rate, the frame, the missing orientation, gravity at rest and a positive yaw rate in a left turn.

File: diffbot_description/urdf/diffbot.urdf.xacro (robot description, xacro)
@@ -1,4 +1,9 @@
 <?xml version="1.0"?>
 <robot xmlns:xacro="http://www.ros.org/wiki/xacro" name="diffbot">
+  <!-- Where the simulation's IMU (imu_link) sits on chassis_link: on the plate, with the board's
+       axes along the robot's (x forward, z up). DiffBot has no IMU on the robot yet; a real one's
+       mounting goes here, or override these, for example imu_xyz:='0 0 0.02' imu_rpy:='0 0 0'. -->
+  <xacro:arg name="imu_xyz" default="0 0 0.01" />
+  <xacro:arg name="imu_rpy" default="0 0 0" />
   <xacro:property name="package_name" value="diffbot_description"/>
   <xacro:property name="robot_name" value="diffbot"/>
@@ -52,4 +57,7 @@
                    enable_gpu="${sensor_prop['laser']['enable_gpu']}">
   </xacro:laser>
+  <xacro:imu_sensor parent_link="chassis_link" sensor_prop="${sensor_prop}">
+    <origin xyz="$(arg imu_xyz)" rpy="$(arg imu_rpy)" />
+  </xacro:imu_sensor>
   <!-- Gazebo -->
   <xacro:gazebo_ros_control robotNamespace="/diffbot">

File: diffbot_description/urdf/include/common_sensors.xacro (robot description, xacro)
@@ -175,22 +175,31 @@
   </gazebo>
 </xacro:macro>
-<xacro:macro name="imu_sensor" params=" *joint_origin parent_link sensor_prop">
-  <xacro:property name="mesh"
-     value="${sensor_prop['imu']['mesh']}"/>
+<!-- IMU: a Bosch BNO055 board, as a small box (sensor_prop['imu']: mass, size, mesh), and a Gazebo
+     IMU sensor that stands in for the real one in the simulation.
+     - imu_link is the sensor's own frame; *origin places it on parent_link, as the board sits on
+       the robot. The real robot's firmware publishes in the same frame (diffbot_base).
+     - The Gazebo plugin (gazebo_plugins' GazeboRosImuSensor, ROS 1) publishes sensor_msgs/Imu on
+       /diffbot/imu/gazebo at 50 Hz, the firmware's rate. Its message includes an orientation that
+       the real sensor doesn't provide, so the simulation passes it through an adapter in
+       diffbot_gazebo, which publishes /diffbot/imu/data_raw like the firmware.
+     - gaussianNoise is one standard deviation that the plugin adds to every value; it's a
+       simulation setting, not the BNO055's measured noise. -->
+<xacro:macro name="imu_sensor" params="parent_link sensor_prop *origin">
+  <xacro:property name="imu" value="${sensor_prop['imu']}"/>
   <link name="imu_link">
-    <xacro:if value="${mesh != '' }" >
-      <visual>
-        <origin xyz="0 0 0" rpy="0 0 0"/>
-        <geometry>
-          <mesh filename="package://${package_name}/meshes/sensors/${mesh}" scale="${sensor_prop['imu']['scale']}" />
+    <xacro:if value="${imu['mesh'] != ''}">
+      <visual>
+        <origin xyz="0 0 0" rpy="0 0 0"/>
+        <geometry>
+          <mesh filename="package://${package_name}/meshes/sensors/${imu['mesh']}" scale="${imu['scale']}"/>
         </geometry>
         <material name="dark_grey"/>
       </visual>
     </xacro:if>
-    <xacro:if value="${mesh == '' }" >
-      <visual>
-        <origin xyz="0 0 0" rpy="0 0 0"/>
-        <geometry>
-          <cylinder radius="${sensor_prop['imu']['radius']}" length="${sensor_prop['imu']['length']}"/>
+    <xacro:if value="${imu['mesh'] == ''}">
+      <visual>
+        <origin xyz="0 0 0" rpy="0 0 0"/>
+        <geometry>
+          <box size="${imu['size']['x']} ${imu['size']['y']} ${imu['size']['z']}"/>
         </geometry>
         <material name="red"/>
@@ -200,45 +209,28 @@
       <origin xyz="0 0 0" rpy="0 0 0"/>
       <geometry>
-        <box size="0.01 0.01 0.01"/>
+        <box size="${imu['size']['x']} ${imu['size']['y']} ${imu['size']['z']}"/>
       </geometry>
     </collision>
-    <xacro:box_inertia m="${sensor_prop['imu']['mass']}"
-                       x="${sensor_prop['imu']['size']['x']}"
-                       y="${sensor_prop['imu']['size']['y']}"
-                       z="${sensor_prop['imu']['size']['y']}" />
-    <!-- Todo delete visual>
-      <origin xyz="0 0 0" rpy="0 0 0"/>
-      <geometry>
-        <box size="0.01 0.01 0.01"/>
-      </geometry>
-    </visual>
-    <inertial>
-      <mass value="1e-5" />
-      <origin xyz="0 0 0" rpy="0 0 0"/>
-      <inertia ixx="1e-6" ixy="0" ixz="0" iyy="1e-6" iyz="0" izz="1e-6" />
-    </inertial-->
+    <xacro:box_inertia m="${imu['mass']}" x="${imu['size']['x']}" y="${imu['size']['y']}" z="${imu['size']['z']}"/>
   </link>
-  <gazebo reference="imu_link">
-    <material>Gazebo/Yellow</material>
-  </gazebo>
   <joint name="imu_joint" type="fixed">
-    <axis xyz="0 1 0" />
-    <xacro:insert_block name="joint_origin" />
     <parent link="${parent_link}"/>
     <child link="imu_link"/>
+    <xacro:insert_block name="origin"/>
   </joint>
   <gazebo reference="imu_link">
-    <sensor type="imu" name="my_imu">
-    <always_on>true</always_on>
-    <!-- Publish at 30 hz -->
-    <update_rate>30</update_rate>
-    <plugin name="my_imu_plugin" filename="libgazebo_ros_imu_sensor.so">
-      <ros>
-        <!-- Will publish to /imu/data -->
-        <namespace>/imu</namespace>
-        <argument>~/out:=data</argument>
-      </ros>
-      <!-- frame_name ommited, will be "my_link" -->
-    </plugin>
+    <sensor type="imu" name="imu">
+      <always_on>true</always_on>
+      <update_rate>50</update_rate>
+      <plugin name="imu_plugin" filename="libgazebo_ros_imu_sensor.so">
+        <robotNamespace>/diffbot</robotNamespace>
+        <topicName>imu/gazebo</topicName>
+        <frameName>imu_link</frameName>
+        <updateRateHZ>50</updateRateHZ>
+        <gaussianNoise>0.005</gaussianNoise>
+        <xyzOffset>0 0 0</xyzOffset>
+        <rpyOffset>0 0 0</rpyOffset>
+        <initialOrientationAsReference>false</initialOrientationAsReference>
+      </plugin>
     </sensor>
   </gazebo>
